Commit message: Added node to create the mujoco xml file, it support mixed input files with file types xml (only mujoco xml), urdf (as file and as string) and xacro. Added a example launch file (without working controllers) to load two different pandas as string from the parameter server, loading a mujoco scene, loading a table and loading a free joint (a cube).

File: panda_mujoco/urdf/dual_panda.urdf.xacro (robot description, xacro)
@@ -52,8 +52,8 @@
     <xacro:property name="world_name" value="world"/>
     <!-- Origin of first arm in the world -->
-    <xacro:property name="origin_xyz_first" value="00 -0.8 0.5"/>
+    <xacro:property name="origin_xyz_first" value="0 -0.8 0.5"/>
     <xacro:property name="origin_rpy_first" value="0 0 1.5708"/>
     <!-- Origin of second arm in the world -->
-    <xacro:property name="origin_xyz_second" value="00 0.8 0.5"/>
+    <xacro:property name="origin_xyz_second" value="0 0.8 0.5"/>
     <xacro:property name="origin_rpy_second" value="0 0 -1.5708"/>
     <!-- Offset of gripper with respect to wrist flange -->
@@ -93,31 +93,4 @@
         <parent link="world"/>
         <child link="table"/>
-        <origin rpy="0 0 0" xyz="0 0 0"/>
-    </joint>
-    <link name="box">
-        <inertial>
-            <origin xyz="0 0 0" rpy="0 0 0"/>
-            <mass value="1"/>
-            <inertia ixx="100"  ixy="0"  ixz="0" iyy="100" iyz="0" izz="100" />
-        </inertial>
-        <visual>
-            <origin xyz="0 0 0.55" rpy="0 0 0" />
-            <geometry>
-                <box size="0.1 0.1 0.1" />
-            </geometry>
-            <material name="Cyan">
-                <color rgba="0 1.0 0.0 1.0"/>
-            </material>
-        </visual>
-        <collision>
-            <origin xyz="0 0 0.55" rpy="0 0 0" />
-            <geometry>
-                <box size="0.1 0.1 0.1" />
-            </geometry>
-        </collision>
-    </link>
-    <joint name="box_table" type="floating">
-        <parent link="table"/>
-        <child link="box"/>
         <origin rpy="0 0 0" xyz="0 0 0"/>
     </joint>

File: panda_mujoco/urdf/panda.urdf.xacro (robot description, xacro)
@@ -1,99 +1,62 @@
 <?xml version="1.0"?>
 <!-- URDF for Franka Emika Panda -->
-<robot xmlns:xacro="http://wiki.ros.org/xacro" name="panda">
+<robot xmlns:xacro="http://wiki.ros.org/xacro">
   <!--                   -->
   <!-- Imported elements -->
   <!--                   -->
-  <xacro:include filename="$(find panda_description)/urdf/panda_arm.xacro"/>
-  <xacro:include filename="$(find panda_description)/urdf/panda_gripper.xacro"/>
-  <xacro:include filename="$(find panda_description)/urdf/panda_utils.xacro"/>
-  <xacro:include filename="$(find panda_mujoco)/urdf/panda.mujoco"/>
-  <!--            -->
-  <!-- Parameters -->
-  <!--            -->
-  <!-- Name of the robot (mandatory) -->
-  <xacro:arg name="name" default="panda"/>
-  <!-- Prefix for all entities -->
-  <xacro:arg name="prefix" default="$(arg name)_"/>
-  <!-- Flag to enable default gripper -->
-  <xacro:arg name="gripper" default="true" />
-  <!-- Flag to enable collision geometry for manipulator's arm -->
-  <xacro:arg name="collision_arm" default="true"/>
-  <!-- Flag to enable collision geometry for manipulator's gripper (hand and fingers) -->
-  <xacro:arg name="collision_gripper" default="true"/>
-  <!-- Flag to enable safety limits controllers on manipulator joints -->
-  <xacro:arg name="safety_limits" default="false"/>
-  <!-- Lower and upper margin for position limits of all safety controllers -->
-  <xacro:arg name="safety_position_margin" default="0.17453293"/>
-  <!-- Parametric k-position factor of all safety controllers -->
-  <xacro:arg name="safety_k_position" default="100.0"/>
-  <!-- Parametric k-velocity factor of all safety controllers -->
-  <xacro:arg name="safety_k_velocity" default="40.0"/>
-  <!-- Flag to enable ros2 controllers for manipulator -->
-  <xacro:arg name="ros2_control" default="true"/>
-  <!-- The ros2_control plugin that should be loaded for the manipulator ('fake', 'ign', 'real' or custom) -->
-  <xacro:arg name="ros2_control_plugin" default="mujoco_ros2_control/MujocoSystem"/>
-  <!-- The output control command interface provided by ros2_control ('position', 'velocity', 'effort' or certain combinations 'position,velocity') -->
-  <xacro:arg name="ros2_control_command_interface" default="effort"/>
-  <!-- The filepath to parameters of ROS 2 controllers -->
-  <xacro:arg name="ros2_controller_parameters" default="$(find panda_mujoco)/config/controllers_$(arg ros2_control_command_interface).yaml"/>
-  <!-- Flag to preserve fixed joints and prevent lumping when generating SDF for Gazebo -->
-  <xacro:arg name="gazebo_preserve_fixed_joint" default="false"/>
-  <!--            -->
-  <!-- Properties -->
-  <!--            -->
-  <!-- Prefixes -->
-  <xacro:property name="prefix_arm" value="$(arg prefix)"/>
-  <xacro:property name="prefix_gripper" value="$(arg prefix)"/>
-  <!-- Origin of arm in the world -->
-  <xacro:property name="world_name" value="world"/>
-  <xacro:property name="origin_xyz" value="0 0 0"/>
-  <xacro:property name="origin_rpy" value="0 0 0"/>
-  <!-- Offset of gripper with respect to wrist flange -->
-  <xacro:property name="gripper_offset_xyz" value="0 0 0"/>
-  <xacro:property name="gripper_offset_rpy" value="0 0 0"/>
-  <!--       -->
-  <!-- Robot -->
-  <!--       -->
-  <!-- Dummy world link that the robot is fixed to -->
-  <xacro:panda_dummy_link
-    link_name="${world_name}"
-    gazebo_preserve_fixed_joint="$(arg gazebo_preserve_fixed_joint)"
-  />
-  <!-- Arm -->
-  <xacro:panda_arm
-    base_parent="world"
-    prefix="${prefix_arm}"
-    origin_xyz="${origin_xyz}"
-    origin_rpy="${origin_rpy}"
-    collision="$(arg collision_arm)"
-    safety_limits="$(arg safety_limits)"
-    safety_position_margin="$(arg safety_position_margin)"
-    safety_k_position="$(arg safety_k_position)"
-    safety_k_velocity="$(arg safety_k_velocity)"
-    ros2_control="$(arg ros2_control)"
-    ros2_control_plugin="$(arg ros2_control_plugin)"
-    ros2_control_command_interface="$(arg ros2_control_command_interface)"
-    gazebo_preserve_fixed_joint="$(arg gazebo_preserve_fixed_joint)"
-  />
-  <!-- Gripper -->
-  <xacro:if value="$(arg gripper)">
-    <xacro:panda_gripper
-      wrist_flange="${prefix_arm}${wrist_flange_name}"
-      prefix="${prefix_gripper}"
-      origin_xyz="${gripper_offset_xyz}"
-      origin_rpy="${gripper_offset_rpy}"
-      collision="$(arg collision_gripper)"
-      ros2_control="$(arg ros2_control)"
-      ros2_control_plugin="$(arg ros2_control_plugin)"
-      ros2_control_command_interface="$(arg ros2_control_command_interface)"
-      gazebo_preserve_fixed_joint="$(arg gazebo_preserve_fixed_joint)"
+  <xacro:macro name="panda" params="name origin_xyz:='0 0 0' origin_rpy:='0 0 0' world_name:=world">
+    <xacro:include filename="$(find panda_description)/urdf/panda_arm.xacro"/>
+    <xacro:include filename="$(find panda_description)/urdf/panda_gripper.xacro"/>
+    <xacro:include filename="$(find panda_description)/urdf/panda_utils.xacro"/>
+    <xacro:include filename="$(find panda_mujoco)/urdf/panda.mujoco"/>
+    <!--            -->
+    <!-- Parameters -->
+    <!--            -->
+    <!-- Prefix for all entities -->
+    <xacro:property name="prefix" value="${name}_"/>
+    <!--       -->
+    <!-- Robot -->
+    <!--       -->
+    <!-- Dummy world link that the robot is fixed to -->
+    <!--xacro:panda_dummy_link
+            link_name="${world_name}"
+            gazebo_preserve_fixed_joint="$(arg gazebo_preserve_fixed_joint)"
+    /-->
+    <!-- Arm -->
+    <xacro:panda_arm
+            base_parent="${world_name}"
+            prefix="${prefix}"
+            origin_xyz="${origin_xyz}"
+            origin_rpy="${origin_rpy}"
+            collision="$(arg collision_arm)"
+            safety_limits="$(arg safety_limits)"
+            safety_position_margin="$(arg safety_position_margin)"
+            safety_k_position="$(arg safety_k_position)"
+            safety_k_velocity="$(arg safety_k_velocity)"
+            ros2_control="$(arg ros2_control)"
+            ros2_control_plugin="$(arg ros2_control_plugin)"
+            ros2_control_command_interface="$(arg ros2_control_command_interface)"
+            gazebo_preserve_fixed_joint="$(arg gazebo_preserve_fixed_joint)"
     />
-  </xacro:if>
-  <!-- Gazebo - ROS 2 control (Ignition) -->
-  <xacro:if value="$(arg ros2_control)">
-    <xacro:if value="${'mujoco' in '$(arg ros2_control_plugin)'}">
-      <xacro:mujoco_ros2_control meshdir="$(find panda_mujoco)/meshes_mujoco/visual"/>
+    <!-- Gripper -->
+    <xacro:if value="$(arg gripper)">
+      <xacro:panda_gripper
+              wrist_flange="${prefix}${wrist_flange_name}"
+              prefix="${prefix}"
+              origin_xyz="0 0 0"
+              origin_rpy="0 0 0"
+              collision="$(arg collision_gripper)"
+              ros2_control="$(arg ros2_control)"
+              ros2_control_plugin="$(arg ros2_control_plugin)"
+              ros2_control_command_interface="$(arg ros2_control_command_interface)"
+              gazebo_preserve_fixed_joint="$(arg gazebo_preserve_fixed_joint)"
+      />
     </xacro:if>
-  </xacro:if>
+    <!-- Gazebo - ROS 2 control (Ignition) -->
+    <xacro:if value="$(arg ros2_control)">
+      <xacro:if value="${'mujoco' in '$(arg ros2_control_plugin)'}">
+        <xacro:mujoco_ros2_control meshdir="$(find panda_mujoco)/meshes_mujoco/visual" prefix="${prefix}"/>
+      </xacro:if>
+    </xacro:if>
+  </xacro:macro>
 </robot>
