Commit message: fixed joints are working but the camera has an issue with the buffer

File: panda_mujoco/urdf/table2.urdf (robot description, URDF)
Before this commit: robot None, 2 links, 1 joints
Links:
- added link camera_link, mass 1; collision box size=0.05 0.05 0.05; visual box size=0.05 0.05 0.05
- link table_base: geometry collision box size=0.758292 1.175997 0.8875; visual mesh filename=file://$(find panda_mujoco)/meshes/table.stl scale=0.001 0.001 0.001
Joints:
- added joint base_to_camera: type fixed, parent base_link, child camera_link, origin xyz=0 0 1.5 rpy=0 0 0
