Commit message: add missing files and added parameter for realtime factor and simulation frequency

File: panda_mujoco/urdf/include/panda_gripper.xacro (robot description, xacro)
@@ -24,5 +24,5 @@
   <xacro:property name="joint_finger1_torque_limit" value="20"/>
   <xacro:property name="joint_finger1_damping" value="3.0"/>
-  <xacro:property name="joint_finger1_friction" value="4"/>
+  <xacro:property name="joint_finger1_friction" value="0.4"/>
   <xacro:property name="link_finger1_name" value="leftfinger"/>
   <xacro:property name="link_finger1_mu" value="1.13"/>
@@ -38,5 +38,5 @@
   <xacro:property name="joint_finger2_torque_limit" value="20"/>
   <xacro:property name="joint_finger2_damping" value="3.0"/>
-  <xacro:property name="joint_finger2_friction" value="4"/>
+  <xacro:property name="joint_finger2_friction" value="0.4"/>
   <xacro:property name="link_finger2_name" value="rightfinger"/>
   <xacro:property name="link_finger2_mu" value="1.13"/>
