Commit message: changed urdf files to use with gazebo ign

File: panda_mujoco/urdf/include/panda.urdf.xacro (robot description, xacro)
@@ -5,5 +5,5 @@
   <!-- Imported elements -->
   <!--                   -->
-  <xacro:macro name="panda" params="name origin_xyz:='0 0 0' origin_rpy:='0 0 0' world_name:=world">
+  <xacro:macro name="panda" params="name origin_xyz:='0 0 0' origin_rpy:='0 0 0' base_parent:=$(arg world_name)">
     <xacro:include filename="$(find panda_mujoco)/urdf/include/panda_arm.xacro"/>
     <xacro:include filename="$(find panda_mujoco)/urdf/include/panda_gripper.xacro"/>
@@ -21,5 +21,5 @@
     <!-- Arm -->
     <xacro:panda_arm
-            base_parent="${world_name}"
+            base_parent="${base_parent}"
             prefix="${prefix}"
             origin_xyz="${origin_xyz}"

File: panda_mujoco/urdf/include/panda_utils.xacro (robot description, xacro)
@@ -22,5 +22,5 @@
         <origin xyz="0 0 0" rpy="${mesh_offset_rpy}"/>
         <geometry>
-          <mesh filename="package://panda_mujoco/meshes/visual/${mesh}.dae"/>
+          <mesh filename="file://$(find panda_mujoco)/meshes/visual/${mesh}.dae"/>
         </geometry>
       </visual>
@@ -29,5 +29,5 @@
           <origin xyz="0 0 0" rpy="${mesh_offset_rpy}"/>
           <geometry>
-            <mesh filename="package://panda_mujoco/meshes/collision/${mesh}.stl"/>
+            <mesh filename="$(find panda_mujoco)/meshes/collision/${mesh}.stl"/>
           </geometry>
         </collision>

File: panda_mujoco/urdf/panda.urdf.xacro (robot description, xacro)
@@ -4,4 +4,5 @@
     <xacro:include filename="$(find panda_mujoco)/urdf/include/panda.urdf.xacro"/>
     <xacro:include filename="$(find panda_mujoco)/urdf/include/panda_utils.xacro"/>
+    <xacro:include filename="$(find panda_mujoco)/urdf/table.urdf.xacro"/>
     <!-- Flag to enable default gripper -->
     <xacro:arg name="gripper" default="true" />
@@ -32,8 +33,14 @@
     <xacro:arg name="mujoco_meshdir" default="$(find panda_mujoco)/meshes/mujoco/visual"/>
     <!-- Dummy world link that the robot is fixed to -->
-    <xacro:panda_dummy_link
+    <!--xacro:panda_dummy_link
             link_name="$(arg world_name)"
             gazebo_preserve_fixed_joint="$(arg gazebo_preserve_fixed_joint)"
-    />
-    <xacro:panda name="$(arg name)" origin_xyz="$(arg origin_xyz)" origin_rpy="$(arg origin_rpy)" world_name="$(arg world_name)"/>
+    /-->
+    <xacro:if value="$(arg generate_world_frame)">
+        <xacro:panda_dummy_link
+            link_name="$(arg world_name)"
+            gazebo_preserve_fixed_joint="$(arg gazebo_preserve_fixed_joint)"
+        />
+    </xacro:if>
+    <xacro:panda name="$(arg name)" origin_xyz="$(arg origin_xyz)" origin_rpy="$(arg origin_rpy)" base_parent="$(arg world_name)"/>
 </robot>
