Commit message: tested gazebo and mujoco launchfiles and removed unused urdf/xacro and config files

File: panda_simulation/urdf/include/panda.urdf.xacro (robot description, xacro)
@@ -6,9 +6,9 @@
   <!--                   -->
   <xacro:macro name="panda" params="name origin_xyz:='0 0 0' origin_rpy:='0 0 0' base_parent:=$(arg world_name)">
-    <xacro:include filename="$(find panda_mujoco)/urdf/include/panda_arm.xacro"/>
-    <xacro:include filename="$(find panda_mujoco)/urdf/include/panda_gripper.xacro"/>
-    <xacro:include filename="$(find panda_mujoco)/urdf/include/panda_utils.xacro"/>
-    <xacro:include filename="$(find panda_mujoco)/config/panda.mujoco"/>
-    <xacro:include filename="$(find panda_mujoco)/config/panda.gazebo"/>
+    <xacro:include filename="$(find panda_simulation)/urdf/include/panda_arm.xacro"/>
+    <xacro:include filename="$(find panda_simulation)/urdf/include/panda_gripper.xacro"/>
+    <xacro:include filename="$(find panda_simulation)/urdf/include/panda_utils.xacro"/>
+    <xacro:include filename="$(find panda_simulation)/config/panda.mujoco"/>
+    <xacro:include filename="$(find panda_simulation)/config/panda.gazebo"/>
     <!--            -->
     <!-- Parameters -->

File: panda_simulation/urdf/include/panda_arm.xacro (robot description, xacro)
@@ -5,6 +5,6 @@
   <!-- Imported elements -->
   <!--                   -->
-  <xacro:include filename="$(find panda_mujoco)/urdf/include/panda_utils.xacro"/>
-  <xacro:include filename="$(find panda_mujoco)/urdf/include/panda.ros2_control"/>
+  <xacro:include filename="$(find panda_simulation)/urdf/include/panda_utils.xacro"/>
+  <xacro:include filename="$(find panda_simulation)/urdf/include/panda.ros2_control"/>
   <!--            -->
   <!-- Properties -->

File: panda_simulation/urdf/include/panda_gripper.xacro (robot description, xacro)
@@ -5,6 +5,6 @@
   <!-- Imported elements -->
   <!--                   -->
-  <xacro:include filename="$(find panda_mujoco)/urdf/include/panda_utils.xacro"/>
-  <xacro:include filename="$(find panda_mujoco)/urdf/include/panda.ros2_control"/>
+  <xacro:include filename="$(find panda_simulation)/urdf/include/panda_utils.xacro"/>
+  <xacro:include filename="$(find panda_simulation)/urdf/include/panda.ros2_control"/>
   <!--            -->
   <!-- Properties -->

File: panda_simulation/urdf/include/panda_utils.xacro (robot description, xacro)
@@ -5,5 +5,5 @@
   <!-- Imported elements -->
   <!--                   -->
-  <xacro:include filename="$(find panda_mujoco)/urdf/include/panda_inertial.xacro"/>
+  <xacro:include filename="$(find panda_simulation)/urdf/include/panda_inertial.xacro"/>
   <!--       -->
   <!-- Macro -->
@@ -22,5 +22,5 @@
         <origin xyz="0 0 0" rpy="${mesh_offset_rpy}"/>
         <geometry>
-          <mesh filename="file://$(find panda_mujoco)/meshes/visual/${mesh}.dae"/>
+          <mesh filename="file://$(find panda_simulation)/meshes/visual/${mesh}.dae"/>
         </geometry>
       </visual>
@@ -29,5 +29,5 @@
           <origin xyz="0 0 0" rpy="${mesh_offset_rpy}"/>
           <geometry>
-            <mesh filename="$(find panda_mujoco)/meshes/collision/${mesh}.stl"/>
+            <mesh filename="$(find panda_simulation)/meshes/collision/${mesh}.stl"/>
           </geometry>
         </collision>

File: panda_simulation/urdf/panda.urdf.xacro (robot description, xacro)
@@ -2,7 +2,7 @@
 <!-- URDF for Franka Emika Panda -->
 <robot xmlns:xacro="http://wiki.ros.org/xacro" name="$(arg name)">
-    <xacro:include filename="$(find panda_mujoco)/urdf/include/panda.urdf.xacro"/>
-    <xacro:include filename="$(find panda_mujoco)/urdf/include/panda_utils.xacro"/>
-    <xacro:include filename="$(find panda_mujoco)/urdf/table2.urdf"/>
+    <xacro:include filename="$(find panda_simulation)/urdf/include/panda.urdf.xacro"/>
+    <xacro:include filename="$(find panda_simulation)/urdf/include/panda_utils.xacro"/>
+    <xacro:include filename="$(find panda_simulation)/urdf/table.urdf"/>
     <!-- Flag to enable default gripper -->
     <xacro:arg name="gripper" default="true" />
@@ -30,6 +30,6 @@
     <!-- Flag to preserve fixed joints and prevent lumping when generating SDF for Gazebo -->
     <xacro:arg name="gazebo_preserve_fixed_joint" default="false"/>
-    <xacro:arg name="ros2_controller_parameters" default="$(find panda_mujoco)/config/controllers_$(arg ros2_control_command_interface).yaml"/>
-    <xacro:arg name="mujoco_meshdir" default="$(find panda_mujoco)/meshes/mujoco/visual"/>
+    <xacro:arg name="ros2_controller_parameters" default="$(find panda_simulation)/config/controllers_$(arg ros2_control_command_interface).yaml"/>
+    <xacro:arg name="mujoco_meshdir" default="$(find panda_simulation)/meshes/mujoco/visual"/>
     <!-- Dummy world link that the robot is fixed to -->
     <!--xacro:panda_dummy_link

File: panda_simulation/urdf/table.urdf (robot description, URDF)
Before this commit: robot table, 6 links, 5 joints
Links:
- removed link leg1_link
- removed link leg2_link
- removed link leg3_link
- removed link leg4_link
- removed link table_top_link
- added link camera_link, mass 1; collision box size=0.05 0.05 0.05; visual box size=0.05 0.05 0.05
- added link table_base, mass 200.0; collision box size=0.758292 1.175997 0.8875; visual mesh filename=file://$(find panda_simulation)/meshes/table.stl scale=0.001 0.001 0.001
Joints:
- removed joint leg1_joint
- removed joint leg2_joint
- removed joint leg3_joint
- removed joint leg4_joint
- removed joint table_top_link_ro_base_link
- added joint base_to_camera: type fixed, parent base_link, child camera_link, origin xyz=0 0 1.5 rpy=0 0 0
- added joint base_to_table_base: type fixed, parent table_base, child base_link, origin xyz=0 0 0 rpy=0 0 0

Commit message: added moveit2 config package

File: panda_simulation/urdf/include/panda.urdf.xacro (robot description, xacro)
@@ -9,6 +9,4 @@
     <xacro:include filename="$(find panda_simulation)/urdf/include/panda_gripper.xacro"/>
     <xacro:include filename="$(find panda_simulation)/urdf/include/panda_utils.xacro"/>
-    <xacro:include filename="$(find panda_simulation)/config/panda.mujoco"/>
-    <xacro:include filename="$(find panda_simulation)/config/panda.gazebo"/>
     <!--            -->
     <!-- Parameters -->
@@ -49,13 +47,4 @@
       />
     </xacro:if>
-    <!-- Gazebo - ROS 2 control (Ignition) -->
-    <xacro:if value="$(arg ros2_control)">
-      <xacro:if value="${'mujoco' in '$(arg ros2_control_plugin)'}">
-        <xacro:mujoco_ros2_control prefix="${prefix}"/>
-      </xacro:if>
-      <xacro:if value="${'ign' in '$(arg ros2_control_plugin)'}">
-        <xacro:ign_ros2_control controller_parameters="$(arg ros2_controller_parameters)"/>
-      </xacro:if>
-    </xacro:if>
   </xacro:macro>
 </robot>

File: panda_simulation/urdf/panda.urdf.xacro (robot description, xacro)
@@ -5,4 +5,6 @@
     <xacro:include filename="$(find panda_simulation)/urdf/include/panda_utils.xacro"/>
     <xacro:include filename="$(find panda_simulation)/urdf/table.urdf"/>
+    <xacro:include filename="$(find panda_simulation)/config/panda.mujoco"/>
+    <xacro:include filename="$(find panda_simulation)/config/panda.gazebo"/>
     <!-- Flag to enable default gripper -->
     <xacro:arg name="gripper" default="true" />
@@ -44,3 +46,5 @@
     </xacro:if>
     <xacro:panda name="$(arg name)" origin_xyz="$(arg origin_xyz)" origin_rpy="$(arg origin_rpy)" base_parent="$(arg world_name)"/>
+    <xacro:mujoco_ros2_control prefix="panda_"/>
+    <xacro:ign_ros2_control/>
 </robot>

File: panda_simulation/urdf/table.urdf (robot description, URDF)
Before this commit: robot None, 3 links, 2 joints
Links:
- link table_base: geometry collision mesh filename=file://$(find panda_simulation)/meshes/table.stl scale=0.001 0.001 0.001; visual mesh filename=file://$(find panda_simulation)/meshes/table.stl scale=0.001 0.001 0.001
