Commit message: used manually generated mjcf file instead of generated

File: panda_simulation/urdf/include/panda_gripper.xacro (robot description, xacro)
@@ -25,5 +25,5 @@
   <xacro:property name="joint_finger1_damping" value="3.0"/>
   <xacro:property name="joint_finger1_friction" value="0.4"/>
-  <xacro:property name="link_finger1_name" value="leftfinger"/>
+  <xacro:property name="link_finger1_name" value="left_finger"/>
   <xacro:property name="link_finger1_mu" value="1.13"/>
   <xacro:property name="link_finger1_mesh_offset" value="0 0 0"/>
@@ -39,5 +39,5 @@
   <xacro:property name="joint_finger2_damping" value="3.0"/>
   <xacro:property name="joint_finger2_friction" value="0.4"/>
-  <xacro:property name="link_finger2_name" value="rightfinger"/>
+  <xacro:property name="link_finger2_name" value="right_finger"/>
   <xacro:property name="link_finger2_mu" value="1.13"/>
   <xacro:property name="link_finger2_mesh_offset" value="0 0 ${pi}"/>

File: panda_simulation/urdf/panda.urdf.xacro (robot description, xacro)
@@ -4,8 +4,7 @@
     <xacro:include filename="$(find panda_simulation)/urdf/include/panda.urdf.xacro"/>
     <xacro:include filename="$(find panda_simulation)/urdf/include/panda_utils.xacro"/>
-    <xacro:include filename="$(find panda_simulation)/urdf/table.urdf"/>
+    <xacro:include filename="$(find panda_simulation)/urdf/table.urdf.xacro"/>
     <xacro:include filename="$(find panda_simulation)/config/panda.mujoco"/>
     <xacro:include filename="$(find panda_simulation)/config/panda.gazebo"/>
-    <xacro:include filename="$(find panda_simulation)/urdf/realsense_d415/_d415.urdf.xacro"/>
     <!-- Flag to enable default gripper -->
     <xacro:arg name="gripper" default="true" />
@@ -34,5 +33,4 @@
     <xacro:arg name="gazebo_preserve_fixed_joint" default="false"/>
     <xacro:arg name="ros2_controller_parameters" default="$(find panda_simulation)/config/controllers_$(arg ros2_control_command_interface).yaml"/>
-    <xacro:arg name="mujoco_meshdir" default="$(find panda_simulation)/meshes/mujoco/visual"/>
     <!-- Dummy world link that the robot is fixed to -->
     <!--xacro:panda_dummy_link
@@ -49,10 +47,3 @@
     <xacro:mujoco_ros2_control prefix="panda_"/>
     <xacro:ign_ros2_control/>
-    <xacro:sensor_d415 parent="$(arg world_name)"
-                       use_nominal_extrinsics="false"
-                       use_mesh="true"
-                       use_mujoco="true"
-                       origin_xyz="0 0 2.5"
-                       origin_rpy="0 1.5708 0">
-    </xacro:sensor_d415>
 </robot>

File: panda_simulation/urdf/realsense_d415/_d415.urdf.xacro (robot description, xacro)
@@ -22,5 +22,5 @@
   <!-- Includes -->
   <xacro:include filename="$(find panda_simulation)/urdf/realsense_d415/_materials.urdf.xacro" />
-  <xacro:macro name="sensor_d415" params="parent origin_xyz='0 0 0' origin_rpy='0 0 0'  name:=camera  use_nominal_extrinsics:=false use_mesh:=true use_mujoco:=false">
+  <xacro:macro name="sensor_d415" params="parent origin_xyz='0 0 0' origin_rpy='0 0 0'  name:=camera  use_nominal_extrinsics:=false use_mesh:=true">
     <xacro:property name="origin_xyz_list" value="${origin_xyz.split()}" />
     <xacro:property name="M_PI" value="3.1415926535897931" />
@@ -72,16 +72,8 @@
         </visual>
         <collision>
-          <xacro:if value="${use_mujoco}">
-            <origin xyz="0 ${-d415_cam_depth_py} 0" rpy="0 0 0"/>
-            <geometry>
-              <box size="${d415_cam_depth} ${d415_cam_width} ${d415_cam_height}"/>
-            </geometry>
-          </xacro:if>
-          <xacro:unless value="${use_mujoco}">
-            <origin xyz="0 ${-d415_cam_depth_py} 0" rpy="0 0 0"/>
-            <geometry>
-              <box size="${d415_cam_depth} ${d415_cam_width} ${d415_cam_height}"/>
-            </geometry>
-          </xacro:unless>
+          <origin xyz="0 ${-d415_cam_depth_py} 0" rpy="0 0 0"/>
+          <geometry>
+            <box size="${d415_cam_depth} ${d415_cam_width} ${d415_cam_height}"/>
+          </geometry>
         </collision>
       <!--/xacro:unless-->
