Commit message: update

File: panda_simulation/urdf/panda.urdf.xacro (robot description, xacro)
@@ -7,4 +7,5 @@
     <xacro:include filename="$(find panda_simulation)/config/panda.mujoco"/>
     <xacro:include filename="$(find panda_simulation)/config/panda.gazebo"/>
+    <xacro:include filename="$(find panda_simulation)/urdf/realsense_d415/_d415.urdf.xacro"/>
     <!-- Flag to enable default gripper -->
     <xacro:arg name="gripper" default="true" />
@@ -48,3 +49,10 @@
     <xacro:mujoco_ros2_control prefix="panda_"/>
     <xacro:ign_ros2_control/>
+    <xacro:sensor_d415 parent="$(arg world_name)"
+                       use_nominal_extrinsics="false"
+                       use_mesh="true"
+                       use_mujoco="true"
+                       origin_xyz="0 0 2.5"
+                       origin_rpy="0 1.5708 0">
+    </xacro:sensor_d415>
 </robot>

File: panda_simulation/urdf/table.urdf (robot description, URDF)
Before this commit: robot None, 3 links, 2 joints
Links:
- removed link camera_link
Joints:
- removed joint base_to_camera
