Commit message: moved sensors to ros2_control instead of spawning nodes by available mujoco sensors

File: examples/franka_mujoco/urdf/ros2_control.urdf.xacro (robot description, xacro)
@@ -49,6 +49,24 @@
       <xacro:if value="${mujoco and ee_id == 'franka_hand'}">
         <xacro:configure_joint joint_name="${arm_id}_finger_joint1" initial_position="0.0" />
-        <!-- Mimiced joints must also be included in ros2_control, then they are mimiced -->
-        <xacro:configure_joint joint_name="${arm_id}_finger_joint2" initial_position="0.0" />
+        <!-- Mimic joints: only state interfaces, no command interfaces -->
+        <joint name="${arm_id}_finger_joint2">
+          <state_interface name="position">
+            <param name="initial_value">0.0</param>
+          </state_interface>
+          <state_interface name="velocity"/>
+          <state_interface name="effort"/>
+        </joint>
+      </xacro:if>
+      <!-- Force/Torque sensor at the end-effector -->
+      <xacro:if value="${mujoco}">
+        <sensor name="${arm_id}_ft_sensor">
+            <param name="site">${arm_id}_link7</param>
+            <state_interface name="force.x"/>
+            <state_interface name="force.y"/>
+            <state_interface name="force.z"/>
+            <state_interface name="torque.x"/>
+            <state_interface name="torque.y"/>
+            <state_interface name="torque.z"/>
+        </sensor>
       </xacro:if>
     </ros2_control>

File: examples/task_table_mujoco/urdf/task_table.urdf.xacro (robot description, xacro)
@@ -2,4 +2,40 @@
 <robot xmlns:xacro="http://ros.org/wiki/xacro" name="task_table">
   <link name="world"/>
+  <!-- ros2_control pose sensors for gear tracking (TF) -->
+  <ros2_control name="TaskTable_Sensors" type="system">
+      <hardware>
+          <plugin>mujoco_ros2_control/MujocoSystem</plugin>
+      </hardware>
+      <sensor name="gears_large_pose">
+          <param name="body">gears_large_link</param>
+          <state_interface name="position.x"/>
+          <state_interface name="position.y"/>
+          <state_interface name="position.z"/>
+          <state_interface name="orientation.x"/>
+          <state_interface name="orientation.y"/>
+          <state_interface name="orientation.z"/>
+          <state_interface name="orientation.w"/>
+      </sensor>
+      <sensor name="gears_medium_pose">
+          <param name="body">gears_medium_link</param>
+          <state_interface name="position.x"/>
+          <state_interface name="position.y"/>
+          <state_interface name="position.z"/>
+          <state_interface name="orientation.x"/>
+          <state_interface name="orientation.y"/>
+          <state_interface name="orientation.z"/>
+          <state_interface name="orientation.w"/>
+      </sensor>
+      <sensor name="gears_small_pose">
+          <param name="body">gears_small_link</param>
+          <state_interface name="position.x"/>
+          <state_interface name="position.y"/>
+          <state_interface name="position.z"/>
+          <state_interface name="orientation.x"/>
+          <state_interface name="orientation.y"/>
+          <state_interface name="orientation.z"/>
+          <state_interface name="orientation.w"/>
+      </sensor>
+  </ros2_control>
   <mujoco>
       <reference name="gears_base_link">

File: examples/unitree_h1_mujoco/urdf/ros2_control.urdf.xacro (robot description, xacro)
@@ -86,4 +86,29 @@
       <!-- <xacro:configure_joint joint_name="R_thumb_intermediate_joint" initial_position="0.0"/> -->
       <!-- <xacro:configure_joint joint_name="R_thumb_distal_joint" initial_position="0.0"/> -->
+      <!-- IMU sensor on torso -->
+      <sensor name="imu_in_torso">
+          <param name="site">imu_in_torso</param>
+          <state_interface name="orientation.x"/>
+          <state_interface name="orientation.y"/>
+          <state_interface name="orientation.z"/>
+          <state_interface name="orientation.w"/>
+          <state_interface name="angular_velocity.x"/>
+          <state_interface name="angular_velocity.y"/>
+          <state_interface name="angular_velocity.z"/>
+          <state_interface name="linear_acceleration.x"/>
+          <state_interface name="linear_acceleration.y"/>
+          <state_interface name="linear_acceleration.z"/>
+      </sensor>
+      <!-- Pose sensor for floating base odometry -->
+      <sensor name="pelvis_pose">
+          <param name="body">pelvis</param>
+          <state_interface name="position.x"/>
+          <state_interface name="position.y"/>
+          <state_interface name="position.z"/>
+          <state_interface name="orientation.x"/>
+          <state_interface name="orientation.y"/>
+          <state_interface name="orientation.z"/>
+          <state_interface name="orientation.w"/>
+      </sensor>
     </ros2_control>
   </xacro:macro>

File: examples/unitree_h1_mujoco/urdf/unitree_h1.urdf.xacro (robot description, xacro)
@@ -65,11 +65,12 @@
             </contact>
             <reference name="torso_link">
-                <site name="torso_link" size="0.01" pos="-0.04452 -0.01891 0.27756" />
+                <site name="imu_in_torso" size="0.01" pos="-0.04452 -0.01891 0.27756" />
             </reference>
             <sensor>
-                <gyro name="test-angular-velocity" site="torso_link" noise="5e-4" cutoff="34.9"/>
-                <accelerometer name="test-linear-acceleration" site="torso_link" noise="1e-2" cutoff="157"/>
+                <gyro name="imu_in_torso-angular-velocity" site="imu_in_torso" noise="5e-4" cutoff="34.9"/>
+                <accelerometer name="imu_in_torso-linear-acceleration" site="imu_in_torso" noise="1e-2" cutoff="157"/>
+                <framequat name="imu_in_torso-orientation" objtype="site" objname="imu_in_torso"/>
                 <framepos name="pelvis_pose" objtype="body" objname="pelvis" reftype="body" refname="world"/>
-                <framequat name="pelvis_quat" objtype="body" objname="pelvis" reftype="body" refname="world"/>
+                <framequat name="pelvis-orientation" objtype="body" objname="pelvis" reftype="body" refname="world"/>
             </sensor>
         </mujoco>
