Commit message: added gl lidar and tests

File: mujoco_ros2_control/test/data/double_pendulum.urdf.xacro (robot description, xacro)
@@ -15,4 +15,6 @@
     <!-- ROS2 Control-->
     <xacro:arg name="command_mode" default="effort" />
+    <!-- disable GL sensors -->
+    <xacro:arg name="with_visual_sensors" default="false" />
   <link name="world" />
   <link name="base_link"/>
@@ -119,4 +121,21 @@
     </sensor>
   </mujoco>
+  <link name="test_camera_link"/>
+  <joint name="world_to_test_camera" type="fixed">
+    <parent link="world"/>
+    <child link="test_camera_link"/>
+    <origin xyz="2.0 0 1.5" rpy="0 0.6 3.14159"/>
+  </joint>
+  <xacro:if value="$(arg with_visual_sensors)">
+    <mujoco>
+      <reference name="test_camera_link">
+        <camera name="test_camera" mode="fixed" fovy="45" quat="0.5 0.5 -0.5 -0.5"/>
+      </reference>
+      <reference name="base_link">
+        <site name="lidar_scan"  size="0.01" pos="0 0 0.6"/>
+        <site name="lidar_cloud" size="0.01" pos="0 0  0.2"/>
+      </reference>
+    </mujoco>
+  </xacro:if>
     <ros2_control name="Unitree_H1_HardwareInterface" type="system">
         <hardware>
@@ -146,4 +165,36 @@
       <xacro:configure_joint joint_name="joint1" initial_position="0.0" command_mode="$(arg command_mode)"/>
       <xacro:configure_joint joint_name="joint2" initial_position="0.0" command_mode="$(arg command_mode)"/>
+      <sensor name="link3_imu">
+        <param name="site">link3</param>
+        <state_interface name="orientation.x"/>
+        <state_interface name="orientation.y"/>
+        <state_interface name="orientation.z"/>
+        <state_interface name="orientation.w"/>
+        <state_interface name="angular_velocity.x"/>
+        <state_interface name="angular_velocity.y"/>
+        <state_interface name="angular_velocity.z"/>
+        <state_interface name="linear_acceleration.x"/>
+        <state_interface name="linear_acceleration.y"/>
+        <state_interface name="linear_acceleration.z"/>
+      </sensor>
+      <sensor name="link3_wrench">
+        <param name="site">link3</param>
+        <state_interface name="force.x"/>
+        <state_interface name="force.y"/>
+        <state_interface name="force.z"/>
+        <state_interface name="torque.x"/>
+        <state_interface name="torque.y"/>
+        <state_interface name="torque.z"/>
+      </sensor>
+      <sensor name="link3_pose">
+        <param name="body">link3</param>
+        <state_interface name="position.x"/>
+        <state_interface name="position.y"/>
+        <state_interface name="position.z"/>
+        <state_interface name="orientation.x"/>
+        <state_interface name="orientation.y"/>
+        <state_interface name="orientation.z"/>
+        <state_interface name="orientation.w"/>
+      </sensor>
     </ros2_control>
 </robot>

Commit message: added camera configuration via parameters (with independent optical and depth frame and configurable fovx, fovy) (legacy camera element is still working)

File: mujoco_ros2_control/test/data/double_pendulum.urdf.xacro (robot description, xacro)
@@ -140,5 +140,14 @@
     <origin xyz="2.0 0 1.5" rpy="0 0.6 3.14159"/>
   </joint>
+  <!-- RealSense D435i from the apt realsense2_description package. Demonstrates a
+       two-frame site camera: color rendered from camera_color_optical_frame,
+       depth from camera_depth_optical_frame (use_nominal_extrinsics gives the
+       real depth<->color parallax). The macro's default name "camera" is renamed
+       to "d435" so the frames are d435_color_optical_frame / d435_depth_optical_frame. -->
   <xacro:if value="$(arg with_visual_sensors)">
+    <xacro:include filename="$(find realsense2_description)/urdf/_d435i.urdf.xacro"/>
+    <xacro:sensor_d435i parent="world" name="d435" use_nominal_extrinsics="true">
+      <origin xyz="1.5 0 0.5" rpy="0 0.3 3.14159"/>
+    </xacro:sensor_d435i>
     <mujoco>
       <reference name="test_camera_link">
@@ -146,6 +155,13 @@
       </reference>
       <reference name="base_link">
-        <site name="lidar_scan"  size="0.01" pos="0 0 0.6"/>
-        <site name="lidar_cloud" size="0.01" pos="0 0  0.2"/>
+        <site name="mjLidar_scan"  size="0.01" pos="0 0 0.6"/>
+        <site name="mjLidar_cloud" size="0.01" pos="0 0  0.2"/>
+      </reference>
+      <!-- Site camera "d435": optical site -> color, depth site -> depth. -->
+      <reference name="d435_color_optical_frame">
+        <site name="mjCamOpt_d435" size="0.01" pos="0 0 0"/>
+      </reference>
+      <reference name="d435_depth_optical_frame">
+        <site name="mjCamDepth_d435" size="0.01" pos="0 0 0"/>
       </reference>
     </mujoco>
