Commit message: feat(examples): add the IMRK table and place the robot on it
The Franka example mounted the arm directly on the ground plane, which does
not match the IMRK lab cell the manipulation scenarios are built around and
leaves no work surface at a realistic height.

Add urdf/imrk_table/imrk_table.urdf.xacro with the lab table mesh, loaded as
an independent scene model via the new load_imrk_table argument (default
true). To place the robot on it, franka.urdf.xacro gains base_xyz / base_rpy
arguments for the world-to-base joint, driven by the new robot_base_xyz launch
argument, and a camera_xyz argument so the scene camera can be raised to match
the new table height instead of being hard-coded at 1 m.

All three xacro arguments default to the previous values, so the description
is unchanged when they are not passed.

Co-Authored-By: Codex <noreply@openai.com>
Co-Authored-By: Claude Opus 5 (1M context) <noreply@anthropic.com>
Co-Authored-By: Adrian Danzglock <adrian.danzglock@dfki.de>

File: mujoco_ros2_control_examples/urdf/franka/franka.urdf.xacro (robot description, xacro)
@@ -18,4 +18,7 @@
     <!-- Franka config -->
     <xacro:arg name="parent" default="world" />
+    <xacro:arg name="base_xyz" default="0 0 0" />
+    <xacro:arg name="base_rpy" default="0 0 0" />
+    <xacro:arg name="camera_xyz" default="1 0 1.0" />
     <xacro:arg name="load_gripper" default="true" />
     <xacro:arg name="ee_id" default="franka_hand" />
@@ -34,5 +37,5 @@
 		<parent link="world" />
 		<child link="base" />
-		<origin rpy="0 0 0" xyz="0 0 0" />
+		<origin rpy="$(arg base_rpy)" xyz="$(arg base_xyz)" />
 	</joint>
     <xacro:include filename="$(find franka_description)/robots/$(arg arm_id)/$(arg arm_id).urdf.xacro" />
@@ -86,5 +89,5 @@
                     camera_name="camera"
                     parent_link="world"
-                    origin_xyz="1 0 1."
+                    origin_xyz="$(arg camera_xyz)"
                     origin_rpy="0 .9 ${pi}">
             </xacro:camera>
