Commit message: add yaro_1105 example

File: mujoco_ros2_control_examples/urdf/franka/franka.urdf.xacro (robot description, xacro)
@@ -2,102 +2,102 @@
 <!-- URDF for Franka Emika Panda -->
 <robot xmlns:xacro="http://wiki.ros.org/xacro" name="$(arg name)">
-    <!-- MuJoCo Config -->
-    <!-- Mujoco compiler options -->
-    <xacro:arg name="mujoco_model_path" default="/tmp/mujoco" />
-    <xacro:arg name="autolimits" default="true" />
-    <xacro:arg name="balanceinertia" default="true" />
-    <!-- Mujoco options -->
-    <xacro:arg name="integrator" default="implicitfast" />
-    <xacro:arg name="gravity" default="0 0 -9.81" />
-    <xacro:arg name="impratio" default="1" />
-    <xacro:arg name="integrator" default="implicitfast" />
-    <xacro:arg name="cone" default="elliptic" />
-    <xacro:arg name="solver" default="Newton" />
-    <xacro:arg name="noslip_iterations" default="3" />
-    <xacro:arg name="multiccd" default="disable" />
-    <!-- Franka config -->
-    <xacro:arg name="parent" default="world" />
-    <xacro:arg name="base_xyz" default="0 0 0" />
-    <xacro:arg name="base_rpy" default="0 0 0" />
-    <xacro:arg name="load_gripper" default="true" />
-    <xacro:arg name="load_realsense" default="true" />
-    <xacro:arg name="render_realsense" default="true" />
-    <!-- Centre of the front-side M6 hole. The 180-degree Y rotation is
+  <!-- MuJoCo Config -->
+  <!-- Mujoco compiler options -->
+  <xacro:arg name="mujoco_model_path" default="/tmp/mujoco" />
+  <xacro:arg name="autolimits" default="true" />
+  <xacro:arg name="balanceinertia" default="true" />
+  <!-- Mujoco options -->
+  <xacro:arg name="integrator" default="implicitfast" />
+  <xacro:arg name="gravity" default="0 0 -9.81" />
+  <xacro:arg name="impratio" default="1" />
+  <xacro:arg name="integrator" default="implicitfast" />
+  <xacro:arg name="cone" default="elliptic" />
+  <xacro:arg name="solver" default="Newton" />
+  <xacro:arg name="noslip_iterations" default="3" />
+  <xacro:arg name="multiccd" default="disable" />
+  <!-- Franka config -->
+  <xacro:arg name="parent" default="world" />
+  <xacro:arg name="base_xyz" default="0 0 0" />
+  <xacro:arg name="base_rpy" default="0 0 0" />
+  <xacro:arg name="load_gripper" default="true" />
+  <xacro:arg name="load_realsense" default="true" />
+  <xacro:arg name="render_realsense" default="true" />
+  <!-- Centre of the front-side M6 hole. The 180-degree Y rotation is
          applied inside the camera-mount macro about the assembly itself;
          rotating this parent frame would swing it through the M6 pivot. -->
-    <xacro:arg name="realsense_xyz" default="0.025 0 0.0075" />
-    <xacro:arg name="realsense_rpy" default="0 0 0" />
-    <xacro:arg name="ee_id" default="franka_hand" />
-    <xacro:arg name="arm_id" default="fp3" />
-    <!-- ROS2 Control-->
-    <xacro:arg name="robot_ip" default="true" />
-    <xacro:arg name="use_fake_hardware" default="false" />
-    <xacro:arg name="fake_sensor_commands" default="false" />
-    <xacro:arg name="mujoco" default="true" />
-    <xacro:arg name="mujoco_effort" default="false" />
-    <!-- Accepted so the launch file can pass it uniformly, but nothing here
+  <xacro:arg name="realsense_xyz" default="0.025 0 0.0075" />
+  <xacro:arg name="realsense_rpy" default="0 0 0" />
+  <xacro:arg name="ee_id" default="franka_hand" />
+  <xacro:arg name="arm_id" default="fp3" />
+  <!-- ROS2 Control-->
+  <xacro:arg name="robot_ip" default="true" />
+  <xacro:arg name="use_fake_hardware" default="false" />
+  <xacro:arg name="fake_sensor_commands" default="false" />
+  <xacro:arg name="mujoco" default="true" />
+  <xacro:arg name="mujoco_effort" default="false" />
+  <!-- Accepted so the launch file can pass it uniformly, but nothing here
          reads it: the GUI window is a simulator setting, and camera rendering no
          longer depends on it. Cameras render offscreen through EGL, which needs
          neither a window nor a display, so a headless run still produces images. -->
-    <xacro:arg name="headless" default="false" />
-    <!-- Import franka urdf file -->
-    <link name="world" />
-	<joint name="world_to_base" type="fixed">
-		<parent link="world" />
-		<child link="base" />
-		<origin rpy="$(arg base_rpy)" xyz="$(arg base_xyz)" />
-	</joint>
-    <xacro:include filename="$(find franka_description)/robots/$(arg arm_id)/$(arg arm_id).urdf.xacro" />
-    <xacro:if value="$(arg load_realsense)">
-        <xacro:include filename="$(find mujoco_ros2_control_examples)/urdf/franka/realsense_d435_wrist.urdf.xacro" />
-        <xacro:franka_realsense_d435_wrist
-            parent="$(arg arm_id)_hand"
-            name="d435"
-            origin_xyz="$(arg realsense_xyz)"
-            origin_rpy="$(arg realsense_rpy)"
-            render_sensors="$(arg render_realsense)" />
-    </xacro:if>
-    <!-- Import franka ros2_control -->
-    <xacro:include filename="$(find mujoco_ros2_control_examples)/urdf/franka/ros2_control.urdf.xacro" />
-    <xacro:franka_arm_ros2_control
+  <xacro:arg name="headless" default="false" />
+  <!-- Import franka urdf file -->
+  <link name="world" />
+  <joint name="world_to_base" type="fixed">
+    <parent link="world" />
+    <child link="base" />
+    <origin rpy="$(arg base_rpy)" xyz="$(arg base_xyz)" />
+  </joint>
+  <xacro:include filename="$(find franka_description)/robots/$(arg arm_id)/$(arg arm_id).urdf.xacro" />
+  <xacro:if value="$(arg load_realsense)">
+    <xacro:include filename="$(find mujoco_ros2_control_examples)/urdf/franka/realsense_d435_wrist.urdf.xacro" />
+    <xacro:franka_realsense_d435_wrist
+      parent="$(arg arm_id)_hand"
+      name="d435"
+      origin_xyz="$(arg realsense_xyz)"
+      origin_rpy="$(arg realsense_rpy)"
+      render_sensors="$(arg render_realsense)" />
+  </xacro:if>
+  <!-- Import franka ros2_control -->
+  <xacro:include filename="$(find mujoco_ros2_control_examples)/urdf/franka/ros2_control.urdf.xacro" />
+  <xacro:franka_arm_ros2_control
+    arm_id="$(arg arm_id)"
+    ee_id="$(arg ee_id)"
+    robot_ip="$(arg robot_ip)"
+    use_fake_hardware="$(arg use_fake_hardware)"
+    fake_sensor_commands="$(arg fake_sensor_commands)"
+    mujoco="$(arg mujoco)"
+    mujoco_effort="$(arg mujoco_effort)"
+    />
+  <!-- Configure mujoco -->
+  <xacro:if value="$(arg mujoco)">
+    <mujoco>
+      <compiler meshdir="$(arg mujoco_model_path)/meshes"
+        discardvisual="false"
+        autolimits="$(arg autolimits)"
+        balanceinertia="$(arg balanceinertia)"
+        />
+      <option integrator="$(arg integrator)"
+        gravity="$(arg gravity)"
+        impratio="$(arg impratio)"
+        cone="$(arg cone)"
+        solver="$(arg solver)"
+        noslip_iterations="$(arg noslip_iterations)">
+        <flag multiccd="$(arg multiccd)"
+          />
+      </option>
+      <!-- Create actuators to use position control -->
+      <xacro:include filename="$(find mujoco_ros2_control_examples)/urdf/franka/mujoco_actuators.urdf.xacro" />
+      <xacro:create_mujoco_actuators
         arm_id="$(arg arm_id)"
         ee_id="$(arg ee_id)"
-        robot_ip="$(arg robot_ip)"
-        use_fake_hardware="$(arg use_fake_hardware)"
-        fake_sensor_commands="$(arg fake_sensor_commands)"
-        mujoco="$(arg mujoco)"
-        mujoco_effort="$(arg mujoco_effort)"
-    />
-    <!-- Configure mujoco -->
-    <xacro:if value="$(arg mujoco)">
-        <mujoco>
-            <compiler meshdir="$(arg mujoco_model_path)/meshes"
-                      discardvisual="false"
-                      autolimits="$(arg autolimits)"
-                      balanceinertia="$(arg balanceinertia)"
-            />
-            <option integrator="$(arg integrator)"
-                    gravity="$(arg gravity)"
-                    impratio="$(arg impratio)"
-                    cone="$(arg cone)"
-                    solver="$(arg solver)"
-                    noslip_iterations="$(arg noslip_iterations)">
-                <flag multiccd="$(arg multiccd)"
-            />
-            </option>
-            <!-- Create actuators to use position control -->
-            <xacro:include filename="$(find mujoco_ros2_control_examples)/urdf/franka/mujoco_actuators.urdf.xacro" />
-            <xacro:create_mujoco_actuators
-                arm_id="$(arg arm_id)"
-                ee_id="$(arg ee_id)"
-            />
-            <reference name="$(arg arm_id)_link7">
-                <site name="$(arg arm_id)_link7" pos="0 0 0.107" quat="0.92388 0 0 -0.382683" />
-            </reference>
-            <sensor>
-                <force name="$(arg arm_id)_link7_force" site="$(arg arm_id)_link7" />
-                <torque name="$(arg arm_id)_link7_torque" site="$(arg arm_id)_link7" />
-            </sensor>
-        </mujoco>
-    </xacro:if>
+        />
+      <reference name="$(arg arm_id)_link7">
+        <site name="$(arg arm_id)_link7" pos="0 0 0.107" quat="0.92388 0 0 -0.382683" />
+      </reference>
+      <sensor>
+        <force name="$(arg arm_id)_link7_force" site="$(arg arm_id)_link7" />
+        <torque name="$(arg arm_id)_link7_torque" site="$(arg arm_id)_link7" />
+      </sensor>
+    </mujoco>
+  </xacro:if>
 </robot>
