Commit message: feat(examples): download the Franka camera mount instead of vendoring it
The D435 wrist mount was Franka's own printable bracket, re-exported through
VTK at 100560 of its 295768 triangles. Franka publishes it in the ZIP that
guide R02241 links, and that archive ships no licence file while the guide
carries only a copyright line, so nothing grants permission to redistribute it
or a derivative of it. Fetch it at configure time behind
DOWNLOAD_FRANKA_CAMERA_MOUNT_ASSET, as the Unitree H1 and IndustReal peg assets
already are, and drop the 5 MB derivative from the tree.

The download URL carries no revision, so it cannot be pinned the way the peg
commit is. Record the archive's SHA256 and warn rather than fail when it stops
matching: a revised mount would move the camera with no other symptom, but a
hard failure would break every build the day Franka republishes.

Convert the mesh to OBJ on the way in. MuJoCo's STL decoder rejects anything
over 200000 faces and the mount is 295768, which is why the vendored copy was
decimated in the first place; the identical triangles load through the OBJ path,
so scripts/stl_to_obj.py welds the triangle soup instead of decimating geometry
the visual origin and its box collision stand-in were measured against. The
result keeps the exact 48 x 60 x 49.95 mm bounds, so no pose changes.

Co-Authored-By: Claude Opus 5 (1M context) <noreply@anthropic.com>

File: mujoco_ros2_control_examples/urdf/franka/realsense_d435_wrist.urdf.xacro (robot description, xacro)
@@ -3,5 +3,10 @@
   <!-- The camera body, its frame tree and its nominal extrinsics all come from
        realsense2_description; only the bracket that bolts it to the Franka Hand
-       is ours, because Franka's printable mount is not part of any ROS package. -->
+       is ours, because Franka's printable mount is not part of any ROS package.
+       The mount mesh itself is not redistributed here - CMakeLists.txt fetches
+       it from franka.de at configure time and rewrites it as an OBJ, because
+       MuJoCo's STL decoder rejects its face count (see
+       ../../meshes/franka/README.md), so it is present only in the install
+       tree, never in the source tree. -->
   <xacro:include filename="$(find realsense2_description)/urdf/_d435.urdf.xacro" />
   <!-- Franka's official D435/D435i wrist mount uses an M6 threaded hole on
@@ -20,10 +25,10 @@
         <origin xyz="0.036 0.030 0" rpy="3.14159265359 3.14159265359 0"/>
         <geometry>
-          <mesh filename="package://mujoco_ros2_control_examples/meshes/franka/realsense_d435/RealSenseD435_Camera_Mount_mujoco.stl"
+          <mesh filename="package://mujoco_ros2_control_examples/meshes/franka/realsense_d435/RealSenseD435_Camera_Mount.obj"
                 scale="0.001 0.001 0.001"/>
         </geometry>
         <material name="realsense_mount_dark_grey"><color rgba="0.18 0.19 0.20 1"/></material>
       </visual>
-      <!-- A simple collision avoids turning a 295k-triangle printable mesh
+      <!-- A simple collision avoids turning the 296k-triangle printable mesh
            into hundreds of convex MuJoCo collision pieces. -->
       <collision>

Commit message: refactor(examples): drop the IndustReal electrical connector task
The task was never renderable as anything better than boxes on trays. IndustReal
builds it from four commercial parts - a Tensility 16-00241 and Qualtek Q-910
plug, a Schurter 4300.0705 and TE 3-213598-2 socket - and NVIDIA identifies them
by part number without redistributing geometry, so upstream ships only the
printable trays. Everything that actually mates was a dimensioned proxy box, and
the proxies did not match the pockets they were supposed to sit in: the 2-prong
plug cradle has its floor 9 mm below the tray rim and spans 61 x 30 mm, while
its proxy was a 28 x 22 x 45 mm box floating 1 mm above the rim. Rather than
keep tuning stand-ins against pockets whose real occupants are unavailable,
remove the task.

This drops the connector_fixture macro, the four fixture instances, the socket
tray lip, the electrical_connectors config block, and the 1.4 MB of tray meshes.
The configured_origin yaw parameter goes with them - it existed only to turn the
2-prong plug tray clear of the gears, and no caller is left.

Also remove meshes/franka/, which held nothing but the camera mount's provenance
note now that the mount itself is downloaded. That note moves into the package
README as "The camera mount mesh", where the rest of the Franka example is
documented, and the comments that pointed at the file follow it.

The gears keep IndustRealKit provenance, so licenses/ and its non-commercial
restriction stay as they are.

Co-Authored-By: Claude Opus 5 (1M context) <noreply@anthropic.com>

File: mujoco_ros2_control_examples/urdf/franka/realsense_d435_wrist.urdf.xacro (robot description, xacro)
@@ -6,7 +6,7 @@
        The mount mesh itself is not redistributed here - CMakeLists.txt fetches
        it from franka.de at configure time and rewrites it as an OBJ, because
-       MuJoCo's STL decoder rejects its face count (see
-       ../../meshes/franka/README.md), so it is present only in the install
-       tree, never in the source tree. -->
+       MuJoCo's STL decoder rejects its face count (see "The camera mount mesh"
+       in ../../README.md), so it is present only in the install tree, never in
+       the source tree. -->
   <xacro:include filename="$(find realsense2_description)/urdf/_d435.urdf.xacro" />
   <!-- Franka's official D435/D435i wrist mount uses an M6 threaded hole on

File: mujoco_ros2_control_examples/urdf/industreal/industreal_task_board.urdf.xacro (robot description, xacro)
@@ -7,6 +7,6 @@
   <xacro:property name="wz" value="${cfg.workspace.xyz[2]}"/>
   <link name="world"/>
-  <xacro:macro name="configured_origin" params="xyz yaw:=0">
-    <origin xyz="${wx + xyz[0]} ${wy + xyz[1]} ${wz + xyz[2]}" rpy="0 0 ${yaw}"/>
+  <xacro:macro name="configured_origin" params="xyz">
+    <origin xyz="${wx + xyz[0]} ${wy + xyz[1]} ${wz + xyz[2]}" rpy="0 0 0"/>
   </xacro:macro>
   <xacro:macro name="inertial" params="mass:=0.1">
@@ -46,41 +46,4 @@
   <xacro:peg_assembly name="rectangular_peg_12mm" shape="rectangular" size="12" fixtures_enabled="${cfg.components.rectangular_peg_12mm.enabled}" object_enabled="${cfg.components.rectangular_peg_12mm.get('object_enabled', cfg.components.rectangular_peg_12mm.enabled)}" pick_xyz="${cfg.components.rectangular_peg_12mm.pick_xyz}" insert_xyz="${cfg.components.rectangular_peg_12mm.insert_xyz}" peg_xyz="${cfg.components.rectangular_peg_12mm.peg_xyz}"/>
   <xacro:peg_assembly name="rectangular_peg_16mm" shape="rectangular" size="16" fixtures_enabled="${cfg.components.rectangular_peg_16mm.enabled}" object_enabled="${cfg.components.rectangular_peg_16mm.get('object_enabled', cfg.components.rectangular_peg_16mm.enabled)}" pick_xyz="${cfg.components.rectangular_peg_16mm.pick_xyz}" insert_xyz="${cfg.components.rectangular_peg_16mm.insert_xyz}" peg_xyz="${cfg.components.rectangular_peg_16mm.peg_xyz}"/>
-  <xacro:macro name="connector_fixture" params="name mesh xyz proxy_size is_pick object_enabled collision_size collision_z socket_z:=0 plug_z:=0 yaw:=0">
-    <link name="${name}_link">
-      <xacro:inertial/>
-      <!-- Exact NVIDIA printable tray; xacro2mjcf marks its surface mesh as
-           shell-inertia while collision remains a stable primitive. -->
-      <visual><geometry><mesh filename="file://$(find mujoco_ros2_control_examples)/meshes/industreal/electrical_connectors/${mesh}"/></geometry><material name="${name}_white"><color rgba="0.92 0.92 0.88 1"/></material></visual>
-      <collision><origin xyz="0 0 ${collision_z}"/><geometry><box size="${collision_size}"/></geometry></collision>
-      <!-- NVIDIA press-fits the socket into the tray and glues the lip on
-           top of it, so socket_z sinks the proxy until its top face is flush
-           with this tray's own top face rather than floating above it. -->
-      <xacro:unless value="${is_pick}"><visual><origin xyz="0 0 ${socket_z}"/><geometry><box size="${proxy_size}"/></geometry><material name="${name}_black"><color rgba="0.025 0.025 0.025 1"/></material></visual></xacro:unless>
-    </link>
-    <joint name="world_to_${name}" type="fixed"><xacro:configured_origin xyz="${xyz}" yaw="${yaw}"/><parent link="world"/><child link="${name}_link"/></joint>
-    <xacro:if value="${is_pick and object_enabled}">
-      <!-- NVIDIA specifies commercial plug part numbers but does not
-           redistribute their meshes. This dimensioned plug is a free body,
-           separate from the exact tray, so it is graspable. plug_z puts it
-           1 mm above its own tray's top face so it starts at rest rather
-           than dropping, the way the gears do; every is_pick fixture must
-           pass it, and it is unused for the insert side. -->
-      <link name="${name}_plug_link">
-        <xacro:inertial mass="0.08"/>
-        <visual><origin xyz="0 0 ${plug_z}"/><geometry><box size="${proxy_size}"/></geometry><material name="${name}_plug_black"><color rgba="0.025 0.025 0.025 1"/></material></visual>
-        <collision><origin xyz="0 0 ${plug_z}"/><geometry><box size="${proxy_size}"/></geometry></collision>
-      </link>
-      <joint name="world_to_${name}_plug" type="floating"><xacro:configured_origin xyz="${xyz}" yaw="${yaw}"/><parent link="world"/><child link="${name}_plug_link"/></joint>
-    </xacro:if>
-  </xacro:macro>
-  <xacro:if value="${cfg.components.electrical_connectors.enabled}">
-    <xacro:property name="connector_objects_enabled" value="${cfg.components.electrical_connectors.get('objects_enabled', cfg.components.electrical_connectors.enabled)}"/>
-    <xacro:connector_fixture name="nema_2_prong_pick" mesh="nema_2-prong_plug_tray.obj" xyz="${cfg.components.electrical_connectors.nema_2_pick_xyz}" proxy_size="0.028 0.022 0.045" is_pick="true" object_enabled="${connector_objects_enabled}" collision_size="0.110 0.080 0.028" collision_z="0.011" plug_z="0.0485" yaw="${pi/2}"/>
-    <xacro:connector_fixture name="nema_2_prong_insert" mesh="nema_2-prong_socket_tray.obj" xyz="${cfg.components.electrical_connectors.nema_2_insert_xyz}" proxy_size="0.030 0.025 0.012" is_pick="false" object_enabled="${connector_objects_enabled}" collision_size="0.070 0.040 0.0315" collision_z="0.01275" socket_z="0.0225"/>
-    <xacro:connector_fixture name="nema_3_prong_pick" mesh="nema_3-prong_plug_tray.obj" xyz="${cfg.components.electrical_connectors.nema_3_pick_xyz}" proxy_size="0.034 0.028 0.050" is_pick="true" object_enabled="${connector_objects_enabled}" collision_size="0.065 0.065 0.029" collision_z="-0.0145" plug_z="0.026"/>
-    <xacro:connector_fixture name="nema_3_prong_insert" mesh="nema_3-prong_socket_tray.obj" xyz="${cfg.components.electrical_connectors.nema_3_insert_xyz}" proxy_size="0.036 0.030 0.012" is_pick="false" object_enabled="${connector_objects_enabled}" collision_size="0.065 0.065 0.0324" collision_z="0.0132" socket_z="0.0234"/>
-    <link name="nema_3_prong_socket_lip_link"><xacro:inertial/><visual><geometry><mesh filename="file://$(find mujoco_ros2_control_examples)/meshes/industreal/electrical_connectors/nema_3-prong_socket_tray_lip.obj"/></geometry><material name="nema_3_lip_white"><color rgba="0.92 0.92 0.88 1"/></material></visual><collision><origin xyz="0 0 0.030"/><geometry><box size="0.044 0.044 0.004"/></geometry></collision></link>
-    <joint name="world_to_nema_3_prong_socket_lip" type="fixed"><xacro:configured_origin xyz="${cfg.components.electrical_connectors.nema_3_insert_xyz}"/><parent link="world"/><child link="nema_3_prong_socket_lip_link"/></joint>
-  </xacro:if>
   <xacro:if value="${cfg.components.gears.enabled}">
     <xacro:mesh_link name="gears_base_link" mesh="industreal/gears/gears_base.stl" color="0.12 0.45 0.25 1" mass="1.0"/>
