Commit message: fix(examples): place the electrical connectors on the IndustReal board
The task board declared all four NEMA fixtures and the README described them as
part of the default layout, but components.electrical_connectors was committed
with enabled: false, so the board came up with only the peg rows and the gears.
Enabling it as-is would have looked wrong, because connector_fixture gave every
tray the same collision primitive (a 75 mm cube at origin z 0.014) while the four
tray meshes do not share an origin convention:

  nema_2-prong_plug_tray     z -0.003 .. +0.025
  nema_2-prong_socket_tray   z -0.003 .. +0.0285
  nema_3-prong_socket_tray   z -0.003 .. +0.0294
  nema_3-prong_plug_tray     z -0.029 ..  0.000

The 3-prong plug tray is modelled below its origin - which is why its configured
z is 0.037 rather than 0.011 - so the shared box sat entirely above its visual
geometry and its plug came to rest on nothing, 28 mm above the visible tray.

Take collision_size and collision_z per fixture from each mesh's own bounding
box, so every tray collides where it is drawn. Add plug_z for the same reason:
the plug proxies were pinned at 0.055, which is 7 mm above the 2-prong tray but
30 mm above the 3-prong one, so place each 1 mm above its own tray's top face
and let it start at rest, the way the loose gears already do.

Verified in MuJoCo: both plugs settle exactly onto their trays, consuming only
the 1 mm clearance (2-prong 0.8860 -> 0.8850, 3-prong 0.9120 -> 0.9110, both to
zero velocity) with no x/y drift from the configured fixture positions.

Co-Authored-By: Claude Opus 5 (1M context) <noreply@anthropic.com>

File: mujoco_ros2_control_examples/urdf/industreal/industreal_task_board.urdf.xacro (robot description, xacro)
@@ -46,5 +46,5 @@
   <xacro:peg_assembly name="rectangular_peg_12mm" shape="rectangular" size="12" fixtures_enabled="${cfg.components.rectangular_peg_12mm.enabled}" object_enabled="${cfg.components.rectangular_peg_12mm.get('object_enabled', cfg.components.rectangular_peg_12mm.enabled)}" pick_xyz="${cfg.components.rectangular_peg_12mm.pick_xyz}" insert_xyz="${cfg.components.rectangular_peg_12mm.insert_xyz}" peg_xyz="${cfg.components.rectangular_peg_12mm.peg_xyz}"/>
   <xacro:peg_assembly name="rectangular_peg_16mm" shape="rectangular" size="16" fixtures_enabled="${cfg.components.rectangular_peg_16mm.enabled}" object_enabled="${cfg.components.rectangular_peg_16mm.get('object_enabled', cfg.components.rectangular_peg_16mm.enabled)}" pick_xyz="${cfg.components.rectangular_peg_16mm.pick_xyz}" insert_xyz="${cfg.components.rectangular_peg_16mm.insert_xyz}" peg_xyz="${cfg.components.rectangular_peg_16mm.peg_xyz}"/>
-  <xacro:macro name="connector_fixture" params="name mesh xyz proxy_size is_pick object_enabled">
+  <xacro:macro name="connector_fixture" params="name mesh xyz proxy_size is_pick object_enabled collision_size collision_z plug_z:=0">
     <link name="${name}_link">
       <xacro:inertial/>
@@ -52,5 +52,5 @@
            shell-inertia while collision remains a stable primitive. -->
       <visual><geometry><mesh filename="file://$(find mujoco_ros2_control_examples)/meshes/industreal/electrical_connectors/${mesh}"/></geometry><material name="${name}_white"><color rgba="0.92 0.92 0.88 1"/></material></visual>
-      <collision><origin xyz="0 0 0.014"/><geometry><box size="0.075 0.075 0.028"/></geometry></collision>
+      <collision><origin xyz="0 0 ${collision_z}"/><geometry><box size="${collision_size}"/></geometry></collision>
       <xacro:unless value="${is_pick}"><visual><origin xyz="0 0 0.034"/><geometry><box size="${proxy_size}"/></geometry><material name="${name}_black"><color rgba="0.025 0.025 0.025 1"/></material></visual></xacro:unless>
     </link>
@@ -59,9 +59,12 @@
       <!-- NVIDIA specifies commercial plug part numbers but does not
            redistribute their meshes. This dimensioned plug is a free body,
-           separate from the exact tray, so it is graspable. -->
+           separate from the exact tray, so it is graspable. plug_z puts it
+           1 mm above its own tray's top face so it starts at rest rather
+           than dropping, the way the gears do; every is_pick fixture must
+           pass it, and it is unused for the insert side. -->
       <link name="${name}_plug_link">
         <xacro:inertial mass="0.08"/>
-        <visual><origin xyz="0 0 0.055"/><geometry><box size="${proxy_size}"/></geometry><material name="${name}_plug_black"><color rgba="0.025 0.025 0.025 1"/></material></visual>
-        <collision><origin xyz="0 0 0.055"/><geometry><box size="${proxy_size}"/></geometry></collision>
+        <visual><origin xyz="0 0 ${plug_z}"/><geometry><box size="${proxy_size}"/></geometry><material name="${name}_plug_black"><color rgba="0.025 0.025 0.025 1"/></material></visual>
+        <collision><origin xyz="0 0 ${plug_z}"/><geometry><box size="${proxy_size}"/></geometry></collision>
       </link>
       <joint name="world_to_${name}_plug" type="floating"><xacro:configured_origin xyz="${xyz}"/><parent link="world"/><child link="${name}_plug_link"/></joint>
@@ -70,8 +73,8 @@
   <xacro:if value="${cfg.components.electrical_connectors.enabled}">
     <xacro:property name="connector_objects_enabled" value="${cfg.components.electrical_connectors.get('objects_enabled', cfg.components.electrical_connectors.enabled)}"/>
-    <xacro:connector_fixture name="nema_2_prong_pick" mesh="nema_2-prong_plug_tray.obj" xyz="${cfg.components.electrical_connectors.nema_2_pick_xyz}" proxy_size="0.028 0.022 0.045" is_pick="true" object_enabled="${connector_objects_enabled}"/>
-    <xacro:connector_fixture name="nema_2_prong_insert" mesh="nema_2-prong_socket_tray.obj" xyz="${cfg.components.electrical_connectors.nema_2_insert_xyz}" proxy_size="0.030 0.025 0.012" is_pick="false" object_enabled="${connector_objects_enabled}"/>
-    <xacro:connector_fixture name="nema_3_prong_pick" mesh="nema_3-prong_plug_tray.obj" xyz="${cfg.components.electrical_connectors.nema_3_pick_xyz}" proxy_size="0.034 0.028 0.050" is_pick="true" object_enabled="${connector_objects_enabled}"/>
-    <xacro:connector_fixture name="nema_3_prong_insert" mesh="nema_3-prong_socket_tray.obj" xyz="${cfg.components.electrical_connectors.nema_3_insert_xyz}" proxy_size="0.036 0.030 0.012" is_pick="false" object_enabled="${connector_objects_enabled}"/>
+    <xacro:connector_fixture name="nema_2_prong_pick" mesh="nema_2-prong_plug_tray.obj" xyz="${cfg.components.electrical_connectors.nema_2_pick_xyz}" proxy_size="0.028 0.022 0.045" is_pick="true" object_enabled="${connector_objects_enabled}" collision_size="0.110 0.080 0.028" collision_z="0.011" plug_z="0.0485"/>
+    <xacro:connector_fixture name="nema_2_prong_insert" mesh="nema_2-prong_socket_tray.obj" xyz="${cfg.components.electrical_connectors.nema_2_insert_xyz}" proxy_size="0.030 0.025 0.012" is_pick="false" object_enabled="${connector_objects_enabled}" collision_size="0.070 0.040 0.0315" collision_z="0.01275"/>
+    <xacro:connector_fixture name="nema_3_prong_pick" mesh="nema_3-prong_plug_tray.obj" xyz="${cfg.components.electrical_connectors.nema_3_pick_xyz}" proxy_size="0.034 0.028 0.050" is_pick="true" object_enabled="${connector_objects_enabled}" collision_size="0.065 0.065 0.029" collision_z="-0.0145" plug_z="0.026"/>
+    <xacro:connector_fixture name="nema_3_prong_insert" mesh="nema_3-prong_socket_tray.obj" xyz="${cfg.components.electrical_connectors.nema_3_insert_xyz}" proxy_size="0.036 0.030 0.012" is_pick="false" object_enabled="${connector_objects_enabled}" collision_size="0.065 0.065 0.0324" collision_z="0.0132"/>
     <link name="nema_3_prong_socket_lip_link"><xacro:inertial/><visual><geometry><mesh filename="file://$(find mujoco_ros2_control_examples)/meshes/industreal/electrical_connectors/nema_3-prong_socket_tray_lip.obj"/></geometry><material name="nema_3_lip_white"><color rgba="0.92 0.92 0.88 1"/></material></visual><collision><origin xyz="0 0 0.030"/><geometry><box size="0.044 0.044 0.004"/></geometry></collision></link>
     <joint name="world_to_nema_3_prong_socket_lip" type="fixed"><xacro:configured_origin xyz="${cfg.components.electrical_connectors.nema_3_insert_xyz}"/><parent link="world"/><child link="nema_3_prong_socket_lip_link"/></joint>

Commit message: fix(examples): stop the connector trays from overlapping each other
Enabling the connector stations put the fixtures where they visibly clipped
through one another. The 2-prong plug tray is the largest fixture on the board
at 110 x 80 mm, but both stations placed pick and insert only 60 mm apart in x,
so it interpenetrated its own socket tray by 30 x 40 x 28 mm; the 3-prong pair,
both 65 mm wide at the same 60 mm spacing, clashed by a further 5 mm.

Right of the gears there are only about 178 mm of free x, and 110 + 65 mm of
tray leaves 9 mm to split between clearing the gears and separating the two
columns - no arrangement of the four positions alone is better than flush. So
give configured_origin an optional yaw (default 0, leaving the pegs and gears
untouched) and turn each station into one column: pick tray behind socket tray
in y, the 2-prong plug tray yawed 90 degrees so its long side runs along y.
That frees 39 mm to distribute, and both stations now clear the gears by 14 mm,
each other by 15 mm, the board edge by 10 mm, and the peg rows by 10 mm.

Also add socket_z. The socket proxies were pinned at 0.034, which floated them
above the 2-prong tray and pushed them 3.2 mm through the 3-prong tray's lip.
NVIDIA press-fits the socket into the tray and glues the lip on top of it, so
sink each proxy until its top face is flush with its own tray's top face.

NVIDIA does not publish fixture positions - the breadboard is a stock Thorlabs
MB3045/M - so the layout is ours to choose; only the mesh footprints are fixed.

Verified against the generated MJCF, walking the body tree with yaw applied:
no connector-to-connector or connector-to-board interpenetration remains except
the lip resting on its own tray, which is the glued joint. Both plugs still
settle 1.0 mm onto their trays to zero velocity at their configured y.

Co-Authored-By: Claude Opus 5 (1M context) <noreply@anthropic.com>

File: mujoco_ros2_control_examples/urdf/industreal/industreal_task_board.urdf.xacro (robot description, xacro)
@@ -7,6 +7,6 @@
   <xacro:property name="wz" value="${cfg.workspace.xyz[2]}"/>
   <link name="world"/>
-  <xacro:macro name="configured_origin" params="xyz">
-    <origin xyz="${wx + xyz[0]} ${wy + xyz[1]} ${wz + xyz[2]}" rpy="0 0 0"/>
+  <xacro:macro name="configured_origin" params="xyz yaw:=0">
+    <origin xyz="${wx + xyz[0]} ${wy + xyz[1]} ${wz + xyz[2]}" rpy="0 0 ${yaw}"/>
   </xacro:macro>
   <xacro:macro name="inertial" params="mass:=0.1">
@@ -46,5 +46,5 @@
   <xacro:peg_assembly name="rectangular_peg_12mm" shape="rectangular" size="12" fixtures_enabled="${cfg.components.rectangular_peg_12mm.enabled}" object_enabled="${cfg.components.rectangular_peg_12mm.get('object_enabled', cfg.components.rectangular_peg_12mm.enabled)}" pick_xyz="${cfg.components.rectangular_peg_12mm.pick_xyz}" insert_xyz="${cfg.components.rectangular_peg_12mm.insert_xyz}" peg_xyz="${cfg.components.rectangular_peg_12mm.peg_xyz}"/>
   <xacro:peg_assembly name="rectangular_peg_16mm" shape="rectangular" size="16" fixtures_enabled="${cfg.components.rectangular_peg_16mm.enabled}" object_enabled="${cfg.components.rectangular_peg_16mm.get('object_enabled', cfg.components.rectangular_peg_16mm.enabled)}" pick_xyz="${cfg.components.rectangular_peg_16mm.pick_xyz}" insert_xyz="${cfg.components.rectangular_peg_16mm.insert_xyz}" peg_xyz="${cfg.components.rectangular_peg_16mm.peg_xyz}"/>
-  <xacro:macro name="connector_fixture" params="name mesh xyz proxy_size is_pick object_enabled collision_size collision_z plug_z:=0">
+  <xacro:macro name="connector_fixture" params="name mesh xyz proxy_size is_pick object_enabled collision_size collision_z socket_z:=0 plug_z:=0 yaw:=0">
     <link name="${name}_link">
       <xacro:inertial/>
@@ -53,7 +53,10 @@
       <visual><geometry><mesh filename="file://$(find mujoco_ros2_control_examples)/meshes/industreal/electrical_connectors/${mesh}"/></geometry><material name="${name}_white"><color rgba="0.92 0.92 0.88 1"/></material></visual>
       <collision><origin xyz="0 0 ${collision_z}"/><geometry><box size="${collision_size}"/></geometry></collision>
-      <xacro:unless value="${is_pick}"><visual><origin xyz="0 0 0.034"/><geometry><box size="${proxy_size}"/></geometry><material name="${name}_black"><color rgba="0.025 0.025 0.025 1"/></material></visual></xacro:unless>
+      <!-- NVIDIA press-fits the socket into the tray and glues the lip on
+           top of it, so socket_z sinks the proxy until its top face is flush
+           with this tray's own top face rather than floating above it. -->
+      <xacro:unless value="${is_pick}"><visual><origin xyz="0 0 ${socket_z}"/><geometry><box size="${proxy_size}"/></geometry><material name="${name}_black"><color rgba="0.025 0.025 0.025 1"/></material></visual></xacro:unless>
     </link>
-    <joint name="world_to_${name}" type="fixed"><xacro:configured_origin xyz="${xyz}"/><parent link="world"/><child link="${name}_link"/></joint>
+    <joint name="world_to_${name}" type="fixed"><xacro:configured_origin xyz="${xyz}" yaw="${yaw}"/><parent link="world"/><child link="${name}_link"/></joint>
     <xacro:if value="${is_pick and object_enabled}">
       <!-- NVIDIA specifies commercial plug part numbers but does not
@@ -68,13 +71,13 @@
         <collision><origin xyz="0 0 ${plug_z}"/><geometry><box size="${proxy_size}"/></geometry></collision>
       </link>
-      <joint name="world_to_${name}_plug" type="floating"><xacro:configured_origin xyz="${xyz}"/><parent link="world"/><child link="${name}_plug_link"/></joint>
+      <joint name="world_to_${name}_plug" type="floating"><xacro:configured_origin xyz="${xyz}" yaw="${yaw}"/><parent link="world"/><child link="${name}_plug_link"/></joint>
     </xacro:if>
   </xacro:macro>
   <xacro:if value="${cfg.components.electrical_connectors.enabled}">
     <xacro:property name="connector_objects_enabled" value="${cfg.components.electrical_connectors.get('objects_enabled', cfg.components.electrical_connectors.enabled)}"/>
-    <xacro:connector_fixture name="nema_2_prong_pick" mesh="nema_2-prong_plug_tray.obj" xyz="${cfg.components.electrical_connectors.nema_2_pick_xyz}" proxy_size="0.028 0.022 0.045" is_pick="true" object_enabled="${connector_objects_enabled}" collision_size="0.110 0.080 0.028" collision_z="0.011" plug_z="0.0485"/>
-    <xacro:connector_fixture name="nema_2_prong_insert" mesh="nema_2-prong_socket_tray.obj" xyz="${cfg.components.electrical_connectors.nema_2_insert_xyz}" proxy_size="0.030 0.025 0.012" is_pick="false" object_enabled="${connector_objects_enabled}" collision_size="0.070 0.040 0.0315" collision_z="0.01275"/>
+    <xacro:connector_fixture name="nema_2_prong_pick" mesh="nema_2-prong_plug_tray.obj" xyz="${cfg.components.electrical_connectors.nema_2_pick_xyz}" proxy_size="0.028 0.022 0.045" is_pick="true" object_enabled="${connector_objects_enabled}" collision_size="0.110 0.080 0.028" collision_z="0.011" plug_z="0.0485" yaw="${pi/2}"/>
+    <xacro:connector_fixture name="nema_2_prong_insert" mesh="nema_2-prong_socket_tray.obj" xyz="${cfg.components.electrical_connectors.nema_2_insert_xyz}" proxy_size="0.030 0.025 0.012" is_pick="false" object_enabled="${connector_objects_enabled}" collision_size="0.070 0.040 0.0315" collision_z="0.01275" socket_z="0.0225"/>
     <xacro:connector_fixture name="nema_3_prong_pick" mesh="nema_3-prong_plug_tray.obj" xyz="${cfg.components.electrical_connectors.nema_3_pick_xyz}" proxy_size="0.034 0.028 0.050" is_pick="true" object_enabled="${connector_objects_enabled}" collision_size="0.065 0.065 0.029" collision_z="-0.0145" plug_z="0.026"/>
-    <xacro:connector_fixture name="nema_3_prong_insert" mesh="nema_3-prong_socket_tray.obj" xyz="${cfg.components.electrical_connectors.nema_3_insert_xyz}" proxy_size="0.036 0.030 0.012" is_pick="false" object_enabled="${connector_objects_enabled}" collision_size="0.065 0.065 0.0324" collision_z="0.0132"/>
+    <xacro:connector_fixture name="nema_3_prong_insert" mesh="nema_3-prong_socket_tray.obj" xyz="${cfg.components.electrical_connectors.nema_3_insert_xyz}" proxy_size="0.036 0.030 0.012" is_pick="false" object_enabled="${connector_objects_enabled}" collision_size="0.065 0.065 0.0324" collision_z="0.0132" socket_z="0.0234"/>
     <link name="nema_3_prong_socket_lip_link"><xacro:inertial/><visual><geometry><mesh filename="file://$(find mujoco_ros2_control_examples)/meshes/industreal/electrical_connectors/nema_3-prong_socket_tray_lip.obj"/></geometry><material name="nema_3_lip_white"><color rgba="0.92 0.92 0.88 1"/></material></visual><collision><origin xyz="0 0 0.030"/><geometry><box size="0.044 0.044 0.004"/></geometry></collision></link>
     <joint name="world_to_nema_3_prong_socket_lip" type="fixed"><xacro:configured_origin xyz="${cfg.components.electrical_connectors.nema_3_insert_xyz}"/><parent link="world"/><child link="nema_3_prong_socket_lip_link"/></joint>
