Commit message: add ulab low level plugin and use both knees for g1 test

File: mujoco_ros2_control_examples/urdf/industreal/industreal_task_board.urdf.xacro (robot description, xacro)
@@ -10,59 +10,321 @@
     <origin xyz="${wx + xyz[0]} ${wy + xyz[1]} ${wz + xyz[2]}" rpy="0 0 0"/>
   </xacro:macro>
-  <xacro:macro name="inertial" params="mass:=0.1">
-    <inertial><origin xyz="0 0 0" rpy="0 0 0"/><mass value="${mass}"/><inertia ixx="0.0001" ixy="0" ixz="0" iyy="0.0001" iyz="0" izz="0.0001"/></inertial>
+  <!--
+    Inertia models:
+      cylinder: solid cylinder, axis along local z
+      box:      solid box with dimensions x, y, z
+      manual:   legacy fallback; replace for dynamic bodies
+    Dimensions and COM offsets are in meters; mass is in kilograms.
+  -->
+  <xacro:macro name="inertial"
+               params="mass:=0.1 shape:=manual
+                       x:=0.01 y:=0.01 z:=0.01
+                       diameter:=0.01 length:=0.05
+                       com_x:=0 com_y:=0 com_z:=0">
+    <inertial>
+      <origin xyz="${com_x} ${com_y} ${com_z}" rpy="0 0 0"/>
+      <mass value="${mass}"/>
+      <!-- Solid cylinder; long axis is local z. -->
+      <xacro:if value="${shape == 'cylinder'}">
+        <inertia
+          ixx="${mass * (3 * (diameter / 2)**2 + length**2) / 12}"
+          ixy="0"
+          ixz="0"
+          iyy="${mass * (3 * (diameter / 2)**2 + length**2) / 12}"
+          iyz="0"
+          izz="${mass * (diameter / 2)**2 / 2}"/>
+      </xacro:if>
+      <!-- Solid rectangular box. -->
+      <xacro:if value="${shape == 'box'}">
+        <inertia
+          ixx="${mass * (y**2 + z**2) / 12}"
+          ixy="0"
+          ixz="0"
+          iyy="${mass * (x**2 + z**2) / 12}"
+          iyz="0"
+          izz="${mass * (x**2 + y**2) / 12}"/>
+      </xacro:if>
+      <!-- Legacy fallback for links without a specified shape. -->
+      <xacro:if value="${shape == 'manual'}">
+        <inertia
+          ixx="0.0001" ixy="0" ixz="0"
+          iyy="0.0001" iyz="0"
+          izz="0.0001"/>
+      </xacro:if>
+    </inertial>
   </xacro:macro>
-  <xacro:macro name="mesh_link" params="name mesh color mass:=0.1">
+  <xacro:macro name="mesh_link"
+               params="name mesh color mass:=0.1
+                       collision_shape:=mesh
+                       inertia_shape:=manual
+                       sx:=0.01 sy:=0.01 sz:=0.01
+                       diameter:=0.01 length:=0.05
+                       com_x:=0 com_y:=0 com_z:=0">
     <link name="${name}">
-      <xacro:inertial mass="${mass}"/>
-      <visual><geometry><mesh filename="file://$(find mujoco_ros2_control_examples)/meshes/${mesh}"/></geometry><material name="${name}_material"><color rgba="${color}"/></material></visual>
-      <collision><geometry><mesh filename="file://$(find mujoco_ros2_control_examples)/meshes/${mesh}"/></geometry></collision>
+      <xacro:inertial
+        mass="${mass}"
+        shape="${inertia_shape}"
+        x="${sx}" y="${sy}" z="${sz}"
+        diameter="${diameter}" length="${length}"
+        com_x="${com_x}" com_y="${com_y}" com_z="${com_z}"/>
+      <visual>
+        <geometry>
+          <mesh filename="file://$(find mujoco_ros2_control_examples)/meshes/${mesh}"/>
+        </geometry>
+        <material name="${name}_material">
+          <color rgba="${color}"/>
+        </material>
+      </visual>
+      <collision>
+      <!-- Solid cylinder; long axis is local z. -->
+      <xacro:if value="${collision_shape == 'cylinder'}">
+        <origin xyz="${com_x} ${com_y} ${com_z}" rpy="0 0 0"/>
+      <geometry>
+        <cylinder radius="${(diameter/2)}" length="${length}"/>
+      </geometry>
+      </xacro:if>
+      <!-- Solid rectangular box. -->
+      <xacro:if value="${collision_shape == 'box'}">
+        <origin xyz="${com_x} ${com_y} ${com_z}" rpy="0 0 0"/>
+      <geometry>
+        <box size="${size * 0.001} ${0.007 if size == 8 else (0.008 if size == 12 else 0.010)} 0.05"/>
+      </geometry>
+      </xacro:if>
+      <!-- Solid rectangular box. -->
+      <xacro:if value="${collision_shape == 'mesh'}">
+      <geometry>
+          <mesh filename="file://$(find mujoco_ros2_control_examples)/meshes/${mesh}"/>
+      </geometry>
+      </xacro:if>
+      </collision>
     </link>
   </xacro:macro>
   <xacro:if value="${cfg.board.enabled}">
     <link name="industreal_breadboard_link">
-      <xacro:inertial mass="12.0"/>
-      <visual><geometry><box size="${str(cfg.board.size[0]) + ' ' + str(cfg.board.size[1]) + ' ' + str(cfg.board.size[2])}"/></geometry><material name="medium_dark_grey"><color rgba="${str(cfg.board.rgba[0]) + ' ' + str(cfg.board.rgba[1]) + ' ' + str(cfg.board.rgba[2]) + ' ' + str(cfg.board.rgba[3])}"/></material></visual>
-      <collision><geometry><box size="${str(cfg.board.size[0]) + ' ' + str(cfg.board.size[1]) + ' ' + str(cfg.board.size[2])}"/></geometry></collision>
+      <xacro:inertial
+        mass="12.0"
+        shape="box"
+        x="${cfg.board.size[0]}"
+        y="${cfg.board.size[1]}"
+        z="${cfg.board.size[2]}"/>
+      <visual>
+        <geometry>
+          <box size="${str(cfg.board.size[0]) + ' ' + str(cfg.board.size[1]) + ' ' + str(cfg.board.size[2])}"/>
+        </geometry>
+        <material name="medium_dark_grey">
+          <color rgba="${str(cfg.board.rgba[0]) + ' ' + str(cfg.board.rgba[1]) + ' ' + str(cfg.board.rgba[2]) + ' ' + str(cfg.board.rgba[3])}"/>
+        </material>
+      </visual>
+      <collision>
+        <geometry>
+          <box size="${str(cfg.board.size[0]) + ' ' + str(cfg.board.size[1]) + ' ' + str(cfg.board.size[2])}"/>
+        </geometry>
+      </collision>
     </link>
-    <joint name="world_to_industreal_breadboard" type="fixed"><xacro:configured_origin xyz="${cfg.board.xyz}"/><parent link="world"/><child link="industreal_breadboard_link"/></joint>
+    <joint name="world_to_industreal_breadboard" type="fixed">
+      <xacro:configured_origin xyz="${cfg.board.xyz}"/>
+      <parent link="world"/>
+      <child link="industreal_breadboard_link"/>
+    </joint>
   </xacro:if>
-  <xacro:macro name="peg_assembly" params="name shape size fixtures_enabled object_enabled pick_xyz insert_xyz peg_xyz">
+  <xacro:macro name="peg_assembly"
+               params="name shape size fixtures_enabled object_enabled pick_xyz insert_xyz peg_xyz">
     <xacro:if value="${fixtures_enabled}">
-      <xacro:mesh_link name="${name}_pick_tray_link" mesh="industreal/pegs/industreal_tray_pick_${shape}_peg_${size}mm.obj" color="0.92 0.92 0.88 1"/>
-      <xacro:mesh_link name="${name}_insert_tray_link" mesh="industreal/pegs/industreal_tray_insert_${shape}_peg_${size}mm.obj" color="0.92 0.92 0.88 1"/>
-      <joint name="world_to_${name}_pick_tray" type="fixed"><xacro:configured_origin xyz="${pick_xyz}"/><parent link="world"/><child link="${name}_pick_tray_link"/></joint>
-      <joint name="world_to_${name}_insert_tray" type="fixed"><xacro:configured_origin xyz="${insert_xyz}"/><parent link="world"/><child link="${name}_insert_tray_link"/></joint>
+      <xacro:mesh_link
+        name="${name}_pick_tray_link"
+        mesh="industreal/pegs/industreal_tray_pick_${shape}_peg_${size}mm.obj"
+        color="0.92 0.92 0.88 1"
+        inertia_shape="box"
+        sx="0.03"
+        sy="0.03"
+        sz="0.03"
+        com_z="0.01"/>
+      <xacro:mesh_link
+        name="${name}_insert_tray_link"
+        mesh="industreal/pegs/industreal_tray_insert_${shape}_peg_${size}mm.obj"
+        color="0.92 0.92 0.88 1"
+        inertia_shape="box"
+        sx="0.03"
+        sy="0.03"
+        sz="0.03"
+        com_z="0.01"/>
+      <joint name="world_to_${name}_pick_tray" type="fixed">
+        <xacro:configured_origin xyz="${pick_xyz}"/>
+        <parent link="world"/>
+        <child link="${name}_pick_tray_link"/>
+      </joint>
+      <joint name="world_to_${name}_insert_tray" type="fixed">
+        <xacro:configured_origin xyz="${insert_xyz}"/>
+        <parent link="world"/>
+        <child link="${name}_insert_tray_link"/>
+      </joint>
     </xacro:if>
     <xacro:if value="${object_enabled}">
-      <xacro:mesh_link name="${name}_link" mesh="industreal/pegs/industreal_${shape}_peg_${size}mm.obj" color="0.68 0.70 0.70 1" mass="0.04"/>
-      <joint name="world_to_${name}" type="floating"><xacro:configured_origin xyz="${peg_xyz}"/><parent link="world"/><child link="${name}_link"/></joint>
+      <!-- Round peg: nominal diameter is size mm; length is 50 mm. -->
+      <xacro:if value="${shape == 'round'}">
+        <xacro:mesh_link
+          name="${name}_link"
+          mesh="industreal/pegs/industreal_${shape}_peg_${size}mm.obj"
+          color="0.68 0.70 0.70 1"
+          mass="0.04"
+          collision_shape="cylinder"
+          inertia_shape="cylinder"
+          diameter="${size * 0.001}"
+          length="0.05"
+          com_z="0.028"/>
+      </xacro:if>
+      <!-- Rectangular KET peg: section dimensions in x/y, length along z. -->
+      <xacro:if value="${shape == 'rectangular'}">
+        <xacro:mesh_link
+          name="${name}_link"
+          mesh="industreal/pegs/industreal_${shape}_peg_${size}mm.obj"
+          color="0.68 0.70 0.70 1"
+          mass="0.04"
+          collision_shape="box"
+          inertia_shape="box"
+          sx="${size * 0.001}"
+          sy="${0.007 if size == 8 else (0.008 if size == 12 else 0.010)}"
+          sz="0.05"
+          com_z="0.028"/>
+      </xacro:if>
+      <joint name="world_to_${name}" type="floating">
+        <xacro:configured_origin xyz="${peg_xyz}"/>
+        <parent link="world"/>
+        <child link="${name}_link"/>
+      </joint>
     </xacro:if>
   </xacro:macro>
-  <xacro:peg_assembly name="round_peg_8mm" shape="round" size="8" fixtures_enabled="${cfg.components.round_peg_8mm.enabled}" object_enabled="${cfg.components.round_peg_8mm.get('object_enabled', cfg.components.round_peg_8mm.enabled)}" pick_xyz="${cfg.components.round_peg_8mm.pick_xyz}" insert_xyz="${cfg.components.round_peg_8mm.insert_xyz}" peg_xyz="${cfg.components.round_peg_8mm.peg_xyz}"/>
-  <xacro:peg_assembly name="round_peg_12mm" shape="round" size="12" fixtures_enabled="${cfg.components.round_peg_12mm.enabled}" object_enabled="${cfg.components.round_peg_12mm.get('object_enabled', cfg.components.round_peg_12mm.enabled)}" pick_xyz="${cfg.components.round_peg_12mm.pick_xyz}" insert_xyz="${cfg.components.round_peg_12mm.insert_xyz}" peg_xyz="${cfg.components.round_peg_12mm.peg_xyz}"/>
-  <xacro:peg_assembly name="round_peg_16mm" shape="round" size="16" fixtures_enabled="${cfg.components.round_peg_16mm.enabled}" object_enabled="${cfg.components.round_peg_16mm.get('object_enabled', cfg.components.round_peg_16mm.enabled)}" pick_xyz="${cfg.components.round_peg_16mm.pick_xyz}" insert_xyz="${cfg.components.round_peg_16mm.insert_xyz}" peg_xyz="${cfg.components.round_peg_16mm.peg_xyz}"/>
-  <xacro:peg_assembly name="rectangular_peg_8mm" shape="rectangular" size="8" fixtures_enabled="${cfg.components.rectangular_peg_8mm.enabled}" object_enabled="${cfg.components.rectangular_peg_8mm.get('object_enabled', cfg.components.rectangular_peg_8mm.enabled)}" pick_xyz="${cfg.components.rectangular_peg_8mm.pick_xyz}" insert_xyz="${cfg.components.rectangular_peg_8mm.insert_xyz}" peg_xyz="${cfg.components.rectangular_peg_8mm.peg_xyz}"/>
-  <xacro:peg_assembly name="rectangular_peg_12mm" shape="rectangular" size="12" fixtures_enabled="${cfg.components.rectangular_peg_12mm.enabled}" object_enabled="${cfg.components.rectangular_peg_12mm.get('object_enabled', cfg.components.rectangular_peg_12mm.enabled)}" pick_xyz="${cfg.components.rectangular_peg_12mm.pick_xyz}" insert_xyz="${cfg.components.rectangular_peg_12mm.insert_xyz}" peg_xyz="${cfg.components.rectangular_peg_12mm.peg_xyz}"/>
-  <xacro:peg_assembly name="rectangular_peg_16mm" shape="rectangular" size="16" fixtures_enabled="${cfg.components.rectangular_peg_16mm.enabled}" object_enabled="${cfg.components.rectangular_peg_16mm.get('object_enabled', cfg.components.rectangular_peg_16mm.enabled)}" pick_xyz="${cfg.components.rectangular_peg_16mm.pick_xyz}" insert_xyz="${cfg.components.rectangular_peg_16mm.insert_xyz}" peg_xyz="${cfg.components.rectangular_peg_16mm.peg_xyz}"/>
+  <xacro:peg_assembly
+    name="round_peg_8mm" shape="round" size="8"
+    fixtures_enabled="${cfg.components.round_peg_8mm.enabled}"
+    object_enabled="${cfg.components.round_peg_8mm.get('object_enabled', cfg.components.round_peg_8mm.enabled)}"
+    pick_xyz="${cfg.components.round_peg_8mm.pick_xyz}"
+    insert_xyz="${cfg.components.round_peg_8mm.insert_xyz}"
+    peg_xyz="${cfg.components.round_peg_8mm.peg_xyz}"/>
+  <xacro:peg_assembly
+    name="round_peg_12mm" shape="round" size="12"
+    fixtures_enabled="${cfg.components.round_peg_12mm.enabled}"
+    object_enabled="${cfg.components.round_peg_12mm.get('object_enabled', cfg.components.round_peg_12mm.enabled)}"
+    pick_xyz="${cfg.components.round_peg_12mm.pick_xyz}"
+    insert_xyz="${cfg.components.round_peg_12mm.insert_xyz}"
+    peg_xyz="${cfg.components.round_peg_12mm.peg_xyz}"/>
+  <xacro:peg_assembly
+    name="round_peg_16mm" shape="round" size="16"
+    fixtures_enabled="${cfg.components.round_peg_16mm.enabled}"
+    object_enabled="${cfg.components.round_peg_16mm.get('object_enabled', cfg.components.round_peg_16mm.enabled)}"
+    pick_xyz="${cfg.components.round_peg_16mm.pick_xyz}"
+    insert_xyz="${cfg.components.round_peg_16mm.insert_xyz}"
+    peg_xyz="${cfg.components.round_peg_16mm.peg_xyz}"/>
+  <xacro:peg_assembly
+    name="rectangular_peg_8mm" shape="rectangular" size="8"
+    fixtures_enabled="${cfg.components.rectangular_peg_8mm.enabled}"
+    object_enabled="${cfg.components.rectangular_peg_8mm.get('object_enabled', cfg.components.rectangular_peg_8mm.enabled)}"
+    pick_xyz="${cfg.components.rectangular_peg_8mm.pick_xyz}"
+    insert_xyz="${cfg.components.rectangular_peg_8mm.insert_xyz}"
+    peg_xyz="${cfg.components.rectangular_peg_8mm.peg_xyz}"/>
+  <xacro:peg_assembly
+    name="rectangular_peg_12mm" shape="rectangular" size="12"
+    fixtures_enabled="${cfg.components.rectangular_peg_12mm.enabled}"
+    object_enabled="${cfg.components.rectangular_peg_12mm.get('object_enabled', cfg.components.rectangular_peg_12mm.enabled)}"
+    pick_xyz="${cfg.components.rectangular_peg_12mm.pick_xyz}"
+    insert_xyz="${cfg.components.rectangular_peg_12mm.insert_xyz}"
+    peg_xyz="${cfg.components.rectangular_peg_12mm.peg_xyz}"/>
+  <xacro:peg_assembly
+    name="rectangular_peg_16mm" shape="rectangular" size="16"
+    fixtures_enabled="${cfg.components.rectangular_peg_16mm.enabled}"
+    object_enabled="${cfg.components.rectangular_peg_16mm.get('object_enabled', cfg.components.rectangular_peg_16mm.enabled)}"
+    pick_xyz="${cfg.components.rectangular_peg_16mm.pick_xyz}"
+    insert_xyz="${cfg.components.rectangular_peg_16mm.insert_xyz}"
+    peg_xyz="${cfg.components.rectangular_peg_16mm.peg_xyz}"/>
   <xacro:if value="${cfg.components.gears.enabled}">
-    <xacro:mesh_link name="gears_base_link" mesh="industreal/gears/gears_base.stl" color="0.12 0.45 0.25 1" mass="1.0"/>
-    <joint name="world_to_gears_base" type="fixed"><xacro:configured_origin xyz="${cfg.components.gears.base_xyz}"/><parent link="world"/><child link="gears_base_link"/></joint>
+    <xacro:mesh_link
+      name="gears_base_link"
+      mesh="industreal/gears/gears_base.stl"
+      color="0.12 0.45 0.25 1"
+      mass="0.1"
+      inertia_shape="box"
+      sx="0.075"
+      sy="0.15"
+      sz="0.01"
+      com_y="-0.007"
+      com_z="-0.01"/>
+    <joint name="world_to_gears_base" type="fixed">
+      <xacro:configured_origin xyz="${cfg.components.gears.base_xyz}"/>
+      <parent link="world"/>
+      <child link="gears_base_link"/>
+    </joint>
   </xacro:if>
   <xacro:if value="${cfg.components.gears.get('objects_enabled', cfg.components.gears.enabled)}">
-    <xacro:mesh_link name="gears_large_link" mesh="industreal/gears/gears_large.stl" color="0.92 0.92 0.88 1" mass="0.04"/>
-    <xacro:mesh_link name="gears_medium_link" mesh="industreal/gears/gears_medium.stl" color="0.92 0.92 0.88 1" mass="0.03"/>
-    <xacro:mesh_link name="gears_small_link" mesh="industreal/gears/gears_small.stl" color="0.92 0.92 0.88 1" mass="0.02"/>
-    <joint name="world_to_gears_large" type="floating"><xacro:configured_origin xyz="${cfg.components.gears.large_xyz}"/><parent link="world"/><child link="gears_large_link"/></joint>
-    <joint name="world_to_gears_medium" type="floating"><xacro:configured_origin xyz="${cfg.components.gears.medium_xyz}"/><parent link="world"/><child link="gears_medium_link"/></joint>
-    <joint name="world_to_gears_small" type="floating"><xacro:configured_origin xyz="${cfg.components.gears.small_xyz}"/><parent link="world"/><child link="gears_small_link"/></joint>
+    <xacro:mesh_link
+      name="gears_large_link"
+      mesh="industreal/gears/gears_large.stl"
+      color="0.92 0.92 0.88 1"
+      mass="0.04"
+      inertia_shape="cylinder"
+      diameter="${cfg.components.gears.large_inertia_diameter}"
+      length="${cfg.components.gears.large_inertia_length}"
+      com_z="0.01"/>
+    <xacro:mesh_link
+      name="gears_medium_link"
+      mesh="industreal/gears/gears_medium.stl"
+      color="0.92 0.92 0.88 1"
+      mass="0.03"
+      inertia_shape="cylinder"
+      diameter="${cfg.components.gears.medium_inertia_diameter}"
+      length="${cfg.components.gears.medium_inertia_length}"/>
+    <xacro:mesh_link
+      name="gears_small_link"
+      mesh="industreal/gears/gears_small.stl"
+      color="0.92 0.92 0.88 1"
+      mass="0.02"
+      inertia_shape="cylinder"
+      diameter="${cfg.components.gears.small_inertia_diameter}"
+      length="${cfg.components.gears.small_inertia_length}"/>
+    <joint name="world_to_gears_large" type="floating">
+      <xacro:configured_origin xyz="${cfg.components.gears.large_xyz}"/>
+      <parent link="world"/>
+      <child link="gears_large_link"/>
+    </joint>
+    <joint name="world_to_gears_medium" type="floating">
+      <xacro:configured_origin xyz="${cfg.components.gears.medium_xyz}"/>
+      <parent link="world"/>
+      <child link="gears_medium_link"/>
+    </joint>
+    <joint name="world_to_gears_small" type="floating">
+      <xacro:configured_origin xyz="${cfg.components.gears.small_xyz}"/>
+      <parent link="world"/>
+      <child link="gears_small_link"/>
+    </joint>
   </xacro:if>
   <mujoco>
-    <default><geom friction="0.5" solimp="0.95 0.99 0.001" solref="0.004 1"/></default>
+    <default>
+      <geom friction="0.5" solimp="0.95 0.99 0.001" solref="0.02 1.5"/>
+    </default>
     <xacro:if value="${cfg.components.gears.get('objects_enabled', cfg.components.gears.enabled)}">
       <sensor>
-        <framepos name="gears_large_pose" objtype="body" objname="gears_large_link" reftype="body" refname="world"/><framequat name="gears_large_quat" objtype="body" objname="gears_large_link" reftype="body" refname="world"/>
-        <framepos name="gears_medium_pose" objtype="body" objname="gears_medium_link" reftype="body" refname="world"/><framequat name="gears_medium_quat" objtype="body" objname="gears_medium_link" reftype="body" refname="world"/>
-        <framepos name="gears_small_pose" objtype="body" objname="gears_small_link" reftype="body" refname="world"/><framequat name="gears_small_quat" objtype="body" objname="gears_small_link" reftype="body" refname="world"/>
+        <framepos
+          name="gears_large_pose"
+          objtype="body" objname="gears_large_link"
+          reftype="body" refname="world"/>
+        <framequat
+          name="gears_large_quat"
+          objtype="body" objname="gears_large_link"
+          reftype="body" refname="world"/>
+        <framepos
+          name="gears_medium_pose"
+          objtype="body" objname="gears_medium_link"
+          reftype="body" refname="world"/>
+        <framequat
+          name="gears_medium_quat"
+          objtype="body" objname="gears_medium_link"
+          reftype="body" refname="world"/>
+        <framepos
+          name="gears_small_pose"
+          objtype="body" objname="gears_small_link"
+          reftype="body" refname="world"/>
+        <framequat
+          name="gears_small_quat"
+          objtype="body" objname="gears_small_link"
+          reftype="body" refname="world"/>
       </sensor>
     </xacro:if>
