Commit message: feat(examples): add the multi-UR example, and fix what it uncovered
ur_multi puts several UR arms in one MuJoCo world under one controller manager.
One description holds them all, so there is a single robot_description, a single
MJCF and a single controller manager; each arm gets its own <ros2_control>
block, and the manager creates one MujocoSystem per block, leaving the arms
independent while they share a physics model.

`ur_types` lists one type per arm, so the row mixes sizes - a ur3e, a ur5e and a
ur10e by default. Each arm is prefixed with its own type, so every joint, frame,
hardware component and controller name says which robot it belongs to; a
repeated type gets an occurrence suffix (ur5e_, ur5e_2_) rather than colliding.
The xacro is the single definition of those prefixes and the launch file reads
them back off the description it generated, so the two cannot drift.

An arm is urdf/ur/ur_arm.urdf.xacro, now shared with the single-arm example, and
the model-wide MuJoCo compiler and solver settings move to
urdf/ur/mujoco_options.urdf.xacro since they may appear only once per model. The
generated ur5e description is unchanged by that refactor.

Fixes this turned up:

* The MuJoCo actuator torque limits were the ur5e row whatever the ur_type,
  despite a comment claiming they mirrored joint_limits.yaml per type. A ur3e
  was allowed 2.8x the shoulder torque it has and a ur10e capped at 45% of its
  own, both silently. They are per type now, with the ur5e-tuned gains scaled
  by torque, so ur.launch.py ur_type:=ur10e is also fixed.
* An example that cannot run built a launch description with no processes, so
  launch_testing reported "Launch stopped before the active tests finished"
  instead of a skip. All five example tests shared this; the description now
  holds a trivial process that keeps the launch alive.
* availability() checked a single asset path and Franka's was None, so the
  example never gated on the assets its description loads unconditionally, and
  every skip message named DOWNLOAD_UNITREE_H1_ASSETS whatever the robot.
* CI checked EGL with `|| true`, so the step verified nothing, and a lost GL
  environment let the GL-gated tests skip while the run stayed green. Both jobs
  now fail on either. The docs claimed CI runs headless and shows a GUI locally,
  neither of which was true.

The README gains the UR and multi-UR examples, with a screenshot of the three
arms alongside their separate hardware components.

File: mujoco_ros2_control_examples/urdf/ur/mujoco_actuators.urdf.xacro (robot description, xacro)
@@ -3,6 +3,10 @@
   <!-- Position + velocity actuator pair for a single UR joint.
        kp/forcerange follow the joint's torque capability; the velocity
-       actuator adds damping for a stable position hold. -->
+       actuator adds damping for a stable position hold.
+       The gains arrive as products, so a whole number would otherwise be written
+       "3000.0"; `tidy` prints it as "3000". Cosmetic - MuJoCo reads either - but
+       it keeps the emitted actuators identical to the hand-written ones. -->
   <xacro:macro name="ur_position_actuator" params="joint effort lower upper kp kv">
+    <xacro:property name="tidy" value="${lambda v: int(v) if float(v).is_integer() else v}"/>
     <position
       name="pos_${joint}"
@@ -10,22 +14,70 @@
       ctrlrange="${lower} ${upper}"
       forcerange="${-effort} ${effort}"
-      kp="${kp}"/>
+      kp="${tidy(kp)}"/>
     <velocity
       name="vel_${joint}"
       joint="${joint}"
       forcerange="${-effort} ${effort}"
-      kv="${kv}"/>
+      kv="${tidy(kv)}"/>
   </xacro:macro>
-  <!-- MuJoCo actuators for the six UR revolute joints.
-       Effort/position limits mirror ur_description/config/<ur_type>/joint_limits.yaml
-       (shoulder + elbow: 150 Nm, wrists: 28 Nm; elbow limited to +-pi). -->
-  <xacro:macro name="create_mujoco_actuators" params="tf_prefix">
+  <!-- max_effort per joint, in ur_description joint order
+       (shoulder_pan, shoulder_lift, elbow, wrist_1, wrist_2, wrist_3), copied
+       from ur_description/config/<ur_type>/joint_limits.yaml. That file cannot
+       be read here: it uses ur_description's own !degrees YAML tag, which the
+       plain loader behind xacro's load_yaml cannot construct.
+       These must be per type. Hard-coding one row - which used to be the case,
+       with the ur5e values - gives a ur3e 2.8x the shoulder torque it has and
+       caps a ur10e at 45% of its own, and both errors are silent. -->
+  <xacro:property name="ur_max_effort" value="${dict(
+      ur3     = [ 56,  56,  28,  12,  12,  12],
+      ur3e    = [ 54,  54,  28,   9,   9,   9],
+      ur5     = [150, 150, 150,  28,  28,  28],
+      ur5e    = [150, 150, 150,  28,  28,  28],
+      ur7e    = [150, 150, 150,  28,  28,  28],
+      ur10    = [330, 330, 150,  56,  56,  56],
+      ur10e   = [330, 330, 150,  54,  54,  54],
+      ur12e   = [330, 330, 150,  54,  54,  54],
+      ur16e   = [330, 330, 150,  54,  54,  54],
+      ur15    = [433, 433, 204,  70,  70,  70],
+      ur18    = [433, 433, 204,  70,  70,  70],
+      ur8long = [433, 433, 204,  70,  70,  70],
+      ur20    = [738, 738, 433, 107, 107, 107],
+      ur30    = [738, 738, 433, 107, 107, 107])}"/>
+  <!-- The gains were tuned on the ur5e, so they are carried to other sizes by
+       scaling with each joint's torque: an arm twice as strong gets twice the
+       stiffness and damping, which keeps the ur5e behaviour bit-for-bit and
+       gives every other type the same hold quality rather than one tuned for a
+       different arm. Reference row: 150 Nm -> kp 3000, kv 200 for the shoulder
+       and elbow; 28 Nm -> kp 500, kv 50 for the wrists. -->
+  <xacro:property name="ur_arm_kp_per_nm" value="${3000.0 / 150.0}"/>
+  <xacro:property name="ur_arm_kv_per_nm" value="${200.0 / 150.0}"/>
+  <xacro:property name="ur_wrist_kp_per_nm" value="${500.0 / 28.0}"/>
+  <xacro:property name="ur_wrist_kv_per_nm" value="${50.0 / 28.0}"/>
+  <!-- MuJoCo actuators for the six UR revolute joints. Position limits mirror
+       ur_description: the elbow is restricted to +-pi, the rest to +-2*pi. -->
+  <xacro:macro name="create_mujoco_actuators" params="tf_prefix ur_type:=ur5e">
+    <!-- An unlisted type falls back to the ur5e row rather than failing the
+         build; check it against joint_limits.yaml before relying on it. -->
+    <xacro:property name="effort"
+                    value="${ur_max_effort.get(ur_type, ur_max_effort['ur5e'])}"/>
     <actuator>
-      <xacro:ur_position_actuator joint="${tf_prefix}shoulder_pan_joint"  effort="150" lower="${-2*pi}" upper="${2*pi}" kp="3000" kv="200"/>
-      <xacro:ur_position_actuator joint="${tf_prefix}shoulder_lift_joint" effort="150" lower="${-2*pi}" upper="${2*pi}" kp="3000" kv="200"/>
-      <xacro:ur_position_actuator joint="${tf_prefix}elbow_joint"         effort="150" lower="${-pi}"   upper="${pi}"   kp="3000" kv="200"/>
-      <xacro:ur_position_actuator joint="${tf_prefix}wrist_1_joint"       effort="28"  lower="${-2*pi}" upper="${2*pi}" kp="500"  kv="50"/>
-      <xacro:ur_position_actuator joint="${tf_prefix}wrist_2_joint"       effort="28"  lower="${-2*pi}" upper="${2*pi}" kp="500"  kv="50"/>
-      <xacro:ur_position_actuator joint="${tf_prefix}wrist_3_joint"       effort="28"  lower="${-2*pi}" upper="${2*pi}" kp="500"  kv="50"/>
+      <xacro:ur_position_actuator joint="${tf_prefix}shoulder_pan_joint"
+        effort="${effort[0]}" lower="${-2*pi}" upper="${2*pi}"
+        kp="${effort[0] * ur_arm_kp_per_nm}" kv="${effort[0] * ur_arm_kv_per_nm}"/>
+      <xacro:ur_position_actuator joint="${tf_prefix}shoulder_lift_joint"
+        effort="${effort[1]}" lower="${-2*pi}" upper="${2*pi}"
+        kp="${effort[1] * ur_arm_kp_per_nm}" kv="${effort[1] * ur_arm_kv_per_nm}"/>
+      <xacro:ur_position_actuator joint="${tf_prefix}elbow_joint"
+        effort="${effort[2]}" lower="${-pi}" upper="${pi}"
+        kp="${effort[2] * ur_arm_kp_per_nm}" kv="${effort[2] * ur_arm_kv_per_nm}"/>
+      <xacro:ur_position_actuator joint="${tf_prefix}wrist_1_joint"
+        effort="${effort[3]}" lower="${-2*pi}" upper="${2*pi}"
+        kp="${effort[3] * ur_wrist_kp_per_nm}" kv="${effort[3] * ur_wrist_kv_per_nm}"/>
+      <xacro:ur_position_actuator joint="${tf_prefix}wrist_2_joint"
+        effort="${effort[4]}" lower="${-2*pi}" upper="${2*pi}"
+        kp="${effort[4] * ur_wrist_kp_per_nm}" kv="${effort[4] * ur_wrist_kv_per_nm}"/>
+      <xacro:ur_position_actuator joint="${tf_prefix}wrist_3_joint"
+        effort="${effort[5]}" lower="${-2*pi}" upper="${2*pi}"
+        kp="${effort[5] * ur_wrist_kp_per_nm}" kv="${effort[5] * ur_wrist_kv_per_nm}"/>
     </actuator>
   </xacro:macro>

File: mujoco_ros2_control_examples/urdf/ur/ur.urdf.xacro (robot description, xacro)
@@ -1,4 +1,5 @@
 <?xml version="1.0"?>
-<!-- URDF for a Universal Robots arm simulated with mujoco_ros2_control -->
+<!-- URDF for a Universal Robots arm simulated with mujoco_ros2_control.
+     The arm itself is ur_arm.urdf.xacro, shared with ur_multi.urdf.xacro. -->
 <robot xmlns:xacro="http://wiki.ros.org/xacro" name="$(arg name)">
     <!-- ============================ Arguments ============================ -->
@@ -22,66 +23,30 @@
     <xacro:arg name="mujoco" default="true"/>
     <xacro:arg name="mujoco_effort" default="false"/>
-    <xacro:property name="tf_prefix" value="$(arg tf_prefix)"/>
-    <!-- ur_description config files for the selected ur_type -->
-    <xacro:property name="ur_type" value="$(arg ur_type)"/>
-    <xacro:property name="ur_config" value="$(find ur_description)/config/${ur_type}"/>
-    <!-- Initial joint configuration (also written as a MuJoCo keyframe via ros2_control). -->
-    <xacro:property name="initial_positions"
-                    value="${dict(
-                        shoulder_pan_joint=0.0,
-                        shoulder_lift_joint=-1.5708,
-                        elbow_joint=1.5708,
-                        wrist_1_joint=-1.5708,
-                        wrist_2_joint=-1.5708,
-                        wrist_3_joint=0.0)}"/>
     <!-- ============================ Robot ============================ -->
     <link name="world"/>
-    <xacro:include filename="$(find ur_description)/urdf/ur_macro.xacro"/>
-    <xacro:ur_robot
+    <xacro:include filename="$(find mujoco_ros2_control_examples)/urdf/ur/ur_arm.urdf.xacro"/>
+    <xacro:ur_arm
         name="$(arg name)"
-        tf_prefix="${tf_prefix}"
+        ur_type="$(arg ur_type)"
+        tf_prefix="$(arg tf_prefix)"
         parent="world"
-        joint_limits_parameters_file="${ur_config}/joint_limits.yaml"
-        kinematics_parameters_file="${ur_config}/default_kinematics.yaml"
-        physical_parameters_file="${ur_config}/physical_parameters.yaml"
-        visual_parameters_file="${ur_config}/visual_parameters.yaml"
-        force_abs_paths="false">
-        <origin xyz="0 0 0" rpy="0 0 0"/>
-    </xacro:ur_robot>
-    <!-- ============================ ros2_control ============================ -->
-    <xacro:include filename="$(find mujoco_ros2_control_examples)/urdf/ur/ros2_control.urdf.xacro"/>
-    <xacro:ur_ros2_control
-        name="UrMujocoSystem"
-        tf_prefix="${tf_prefix}"
+        xyz="0 0 0"
+        rpy="0 0 0"
         mujoco="$(arg mujoco)"
-        mujoco_effort="$(arg mujoco_effort)"
-        initial_positions="${initial_positions}"/>
+        mujoco_effort="$(arg mujoco_effort)"/>
     <!-- ============================ MuJoCo config ============================ -->
     <xacro:if value="$(arg mujoco)">
-        <mujoco>
-            <compiler meshdir="$(arg mujoco_model_path)/meshes"
-                      discardvisual="false"
-                      autolimits="$(arg autolimits)"
-                      balanceinertia="$(arg balanceinertia)"/>
-            <option integrator="$(arg integrator)"
-                    gravity="$(arg gravity)"
-                    impratio="$(arg impratio)"
-                    cone="$(arg cone)"
-                    solver="$(arg solver)"
-                    noslip_iterations="$(arg noslip_iterations)">
-                <flag multiccd="$(arg multiccd)"/>
-            </option>
-            <!-- Position actuators -->
-            <xacro:include filename="$(find mujoco_ros2_control_examples)/urdf/ur/mujoco_actuators.urdf.xacro"/>
-            <xacro:create_mujoco_actuators tf_prefix="${tf_prefix}"/>
-            <!-- Wrist force/torque sensor -->
-            <reference name="${tf_prefix}wrist_3_link">
-                <site name="${tf_prefix}tcp_ft_site" pos="0 0.1 0" quat="1 0 0 0"/>
-            </reference>
-            <sensor>
-                <force name="${tf_prefix}tcp_ft_force" site="${tf_prefix}tcp_ft_site"/>
-                <torque name="${tf_prefix}tcp_ft_torque" site="${tf_prefix}tcp_ft_site"/>
-            </sensor>
-        </mujoco>
+        <xacro:include filename="$(find mujoco_ros2_control_examples)/urdf/ur/mujoco_options.urdf.xacro"/>
+        <xacro:ur_mujoco_options
+            mujoco_model_path="$(arg mujoco_model_path)"
+            autolimits="$(arg autolimits)"
+            balanceinertia="$(arg balanceinertia)"
+            integrator="$(arg integrator)"
+            gravity="$(arg gravity)"
+            impratio="$(arg impratio)"
+            cone="$(arg cone)"
+            solver="$(arg solver)"
+            noslip_iterations="$(arg noslip_iterations)"
+            multiccd="$(arg multiccd)"/>
     </xacro:if>
 </robot>
