Commit message: fix(examples): correct G1 ankle crank geometry and retune loop/gains
Two real modeling bugs in the parallel-ankle mechanism, not just
placeholder values:

- Motor axis was local Y; the CAD assembly (unitree_ankle.blend,
  joint_motor_1/joint_motor_b) has it on local X. The crank visual/
  collision was also a fixed 15mm stub along local X rather than a
  cylinder actually running from the joint origin to the measured
  swing_xyz tip (now crank_mid/crank_rpy/crank_len, precomputed per rod).
- The rodA/B_loop equality constraints used solref "0.001 1" - a
  timeconst equal to the sim's own 1ms step, leaving essentially no
  numerical margin, so crank PD feedback resonated into divergence
  within ~1s under real ankle load. Raising the damping ratio (1 -> 3)
  fixes the resonance without the ~100x stiffness loss raising
  timeconst alone would cause. Separately, the motor_joint effort limit
  (20 N*m) was well below the ~33 N*m this linkage's Jacobian requires
  to match Unitree's own 35 N*m ankle_pitch/roll rating, so the PD was
  saturating and behaving like a relay near the standing pose.

With the corrected geometry, the loop-closure initial positions in
ros2_control.urdf.xacro and hold_start_message_ab.yaml no longer match
reality, so they're re-solved via a 3-equation/3-unknown FK root-find
(closing each rod's loop at the ankle's own -0.2/0.0 initial pose)
rather than hand-tuned, and hold_start_message_ab's kp/kd is retuned to
100/4 (from a 20/0.5 placeholder) via an offline load+disturbance sweep
against the corrected geometry.

File: mujoco_ros2_control_examples/urdf/unitree_g1/ros2_control.urdf.xacro (robot description, xacro)
@@ -56,16 +56,24 @@
         </xacro:if>
       </xacro:macro>
-      <xacro:g1_passive_joint name="left_rodA_motor_joint"  initial_position="-0.5596"/>
-      <xacro:g1_passive_joint name="left_rodB_motor_joint"  initial_position="-0.3058"/>
-      <xacro:g1_passive_joint name="right_rodA_motor_joint" initial_position="-0.5596"/>
-      <xacro:g1_passive_joint name="right_rodB_motor_joint" initial_position="-0.3058"/>
-      <xacro:g1_passive_joint name="left_rodA_swing1_joint"  initial_position="-0.3690"/>
-      <xacro:g1_passive_joint name="left_rodA_swing2_joint"  initial_position="0.3866"/>
-      <xacro:g1_passive_joint name="left_rodB_swing1_joint"  initial_position="-0.1927"/>
-      <xacro:g1_passive_joint name="left_rodB_swing2_joint"  initial_position="0.2985"/>
-      <xacro:g1_passive_joint name="right_rodA_swing1_joint" initial_position="0.3690"/>
-      <xacro:g1_passive_joint name="right_rodA_swing2_joint" initial_position="0.3866"/>
-      <xacro:g1_passive_joint name="right_rodB_swing1_joint" initial_position="0.1927"/>
-      <xacro:g1_passive_joint name="right_rodB_swing2_joint" initial_position="0.2985"/>
+      <!-- Solved (not hand-tuned): the crank/swing angles that close each
+           rod's loop-closure constraint (rod tip == its ankle_roll_link
+           plate site) with left/right_ankle_pitch/roll_joint sitting at
+           their own initial pose (-0.2/0.0), via a 3-equation/3-unknown
+           forward-kinematics root-find in the corrected geometry (motor
+           axis local X, tightened swing_rpy - see unitree_g1.urdf.xacro's
+           unitree_g1_ankle_rod macro). Re-solve if revolute_xyz/swing_xyz/
+           swing_rpy/rod_length or the ankle's own initial_position change. -->
+      <xacro:g1_passive_joint name="left_rodA_motor_joint"  initial_position="0.275878"/>
+      <xacro:g1_passive_joint name="left_rodB_motor_joint"  initial_position="-0.280022"/>
+      <xacro:g1_passive_joint name="right_rodA_motor_joint" initial_position="-0.275878"/>
+      <xacro:g1_passive_joint name="right_rodB_motor_joint" initial_position="0.280022"/>
+      <xacro:g1_passive_joint name="left_rodA_swing1_joint"  initial_position="0.221627"/>
+      <xacro:g1_passive_joint name="left_rodA_swing2_joint"  initial_position="0.168432"/>
+      <xacro:g1_passive_joint name="left_rodB_swing1_joint"  initial_position="-0.246636"/>
+      <xacro:g1_passive_joint name="left_rodB_swing2_joint"  initial_position="-0.137527"/>
+      <xacro:g1_passive_joint name="right_rodA_swing1_joint" initial_position="-0.221627"/>
+      <xacro:g1_passive_joint name="right_rodA_swing2_joint" initial_position="0.168432"/>
+      <xacro:g1_passive_joint name="right_rodB_swing1_joint" initial_position="0.246636"/>
+      <xacro:g1_passive_joint name="right_rodB_swing2_joint" initial_position="-0.137527"/>
       <!-- Waist (kp = base*5.0: yaw 1000, roll/pitch 200) -->
       <xacro:g1_joint name="waist_yaw_joint"   kp="1000" kd="5" initial_position="0.0"/>

File: mujoco_ros2_control_examples/urdf/unitree_g1/unitree_g1.urdf.xacro (robot description, xacro)
@@ -26,22 +26,27 @@
   <!-- ==================== Optional parallel ankle mechanism ==================== -->
   <xacro:macro name="unitree_g1_ankle_rod"
-               params="suffix knee_link revolute_xyz swing_xyz swing_rpy rod_length">
+               params="suffix knee_link revolute_xyz swing_xyz swing_rpy rod_length crank_mid crank_rpy crank_len">
     <!-- The real motor: a revolute joint on the shank driving a short, fixed
          crank arm (measured from the real CAD assembly, unitree_ankle.blend/
          G1 ankle STEP - see swing_xyz below for the tip offset, which is not
-         purely radial) whose tip is where the connecting rod attaches. -->
+         purely radial) whose tip is where the connecting rod attaches.
+         The crank_link visual/collision cylinder below runs from the joint
+         origin out to that measured tip (crank_mid/crank_rpy/crank_len,
+         precomputed so the cylinder's own Z-axis lands exactly on
+         swing_xyz) - previously this was a fixed 15mm stub along local X
+         that did not represent the true crank geometry. -->
     <link name="${suffix}_crank_link">
       <inertial>
         <mass value="0.05"/>
-        <origin xyz="0.0075 0 0" rpy="0 0 0"/>
+        <origin xyz="${crank_mid}" rpy="0 0 0"/>
         <inertia ixx="1e-6" iyy="1e-6" izz="1e-6" ixy="0" ixz="0" iyz="0"/>
       </inertial>
       <visual>
-        <origin xyz="0.0075 0 0" rpy="0 1.5707963267948966 0"/>
-        <geometry><cylinder radius="0.001" length="0.015"/></geometry>
+        <origin xyz="${crank_mid}" rpy="${crank_rpy}"/>
+        <geometry><cylinder radius="0.0015" length="${crank_len}"/></geometry>
       </visual>
       <collision>
-        <origin xyz="0.0075 0 0" rpy="0 1.5707963267948966 0"/>
-        <geometry><cylinder radius="0.001" length="0.015"/></geometry>
+        <origin xyz="${crank_mid}" rpy="${crank_rpy}"/>
+        <geometry><cylinder radius="0.0015" length="${crank_len}"/></geometry>
       </collision>
     </link>
@@ -50,10 +55,23 @@
       <child link="${suffix}_crank_link"/>
       <origin xyz="${revolute_xyz}" rpy="0 0 0"/>
-      <axis xyz="0 1 0"/>
+      <!-- Axis measured/verified directly in the CAD assembly
+           (unitree_ankle.blend, joint_motor_1/joint_motor_b) as local X -
+           not Y, which this used to be set to. -->
+      <axis xyz="1 0 0"/>
       <!-- Real range measured from Unitree's own G1 ankle demo (A/B motor
            telemetry sweeps roughly -0.67..+0.97 / -0.6..+0.57 rad) - the
            15mm-crank-arm placeholder this used to be tuned against only
-           supported +-0.5 rad and could not reach a normal standing pose. -->
-      <limit lower="-0.8" upper="1.1" effort="20" velocity="10"/>
+           supported +-0.5 rad and could not reach a normal standing pose.
+           effort raised from a 20 N*m placeholder to 35: Unitree's own
+           g1_29dof_rev_1_0.urdf rates left/right_ankle_pitch/roll_joint at
+           35 N*m each (the ankle-output torque, since that URDF models the
+           ankle as a plain 2-DOF joint rather than this parallel linkage).
+           Converting that through this linkage's Jacobian at the standing
+           pose (d(ankle_pitch,roll)/d(motor_A,motor_B)) gives ~33 N*m of
+           required crank torque to reach the same ankle-output envelope -
+           20 N*m was saturating well before that, which was a real
+           contributor to both the standing droop and the PD oscillation
+           (a torque-clamped PD behaves like a relay near saturation). -->
+      <limit lower="-0.8" upper="1.1" effort="35" velocity="10"/>
       <dynamics damping="3.0" friction="0.05"/>
     </joint>
@@ -64,4 +82,8 @@
         <inertia ixx="1e-7" iyy="1e-7" izz="1e-7" ixy="0" ixz="0" iyz="0"/>
       </inertial>
+      <visual>
+        <origin xyz="0 0 0" rpy="0 0 0"/>
+        <geometry><sphere radius="0.003"/></geometry>
+      </visual>
     </link>
     <joint name="${suffix}_swing1_joint" type="continuous">
@@ -77,4 +99,8 @@
         <inertia ixx="1e-7" iyy="1e-7" izz="1e-7" ixy="0" ixz="0" iyz="0"/>
       </inertial>
+      <visual>
+        <origin xyz="0 0 0" rpy="0 0 0"/>
+        <geometry><sphere radius="0.003"/></geometry>
+      </visual>
     </link>
     <joint name="${suffix}_swing2_joint" type="continuous">
@@ -113,14 +139,18 @@
     <xacro:unitree_g1_ankle_rod suffix="left_rodA" knee_link="left_knee_link"
         revolute_xyz="0.028017 0.0000816 -0.149261" swing_xyz="0.007631 0.016661 -0.003724"
-        swing_rpy="3.10071807 -0.11497669 -2.45906242" rod_length="0.157021"/>
+        swing_rpy="3.09582687 -0.07460496 -2.4608202" rod_length="0.157021"
+        crank_mid="0.003815 0.008330 -0.001862" crank_rpy="-1.790698 0.420345 -0.520459" crank_len="0.018700"/>
     <xacro:unitree_g1_ankle_rod suffix="left_rodB" knee_link="left_knee_link"
         revolute_xyz="0.029387 0.0001696 -0.084324" swing_xyz="0.014715 -0.016386 -0.00465"
-        swing_rpy="3.12888053 -0.04891438 -2.63316226" rod_length="0.221363"/>
+        swing_rpy="3.08875477 -0.0844462 -2.63199475" rod_length="0.221363"
+        crank_mid="0.007358 -0.008193 -0.002325" crank_rpy="1.847306 0.712515 0.915153" crank_len="0.022509"/>
     <xacro:unitree_g1_ankle_rod suffix="right_rodA" knee_link="right_knee_link"
         revolute_xyz="0.028017 -0.0000816 -0.149261" swing_xyz="0.007631 -0.016661 -0.003724"
-        swing_rpy="-3.10071807 -0.11497669 2.45906242" rod_length="0.157021"/>
+        swing_rpy="-3.09582687 -0.07460496 2.4608202" rod_length="0.157021"
+        crank_mid="0.003815 -0.008330 -0.001862" crank_rpy="1.790698 0.420345 0.520459" crank_len="0.018700"/>
     <xacro:unitree_g1_ankle_rod suffix="right_rodB" knee_link="right_knee_link"
         revolute_xyz="0.029387 -0.0001696 -0.084324" swing_xyz="0.014715 0.016386 -0.00465"
-        swing_rpy="-3.12888053 -0.04891438 2.63316226" rod_length="0.221363"/>
+        swing_rpy="-3.08875477 -0.0844462 2.63199475" rod_length="0.221363"
+        crank_mid="0.007358 0.008193 -0.002325" crank_rpy="-1.847306 0.712515 -0.915153" crank_len="0.022509"/>
   </xacro:if>
   <!-- ROS optical frame for the d435 depth camera (REP-103: x-right, y-down, z-forward) -->
@@ -222,8 +252,8 @@
         <reference name="right_ankle_roll_link"><site name="right_rodB_plate_target" pos="0.022123 0.015012 0.008328" size="0.003"/></reference>
         <equality>
-          <connect name="left_rodA_loop" site1="left_rodA_rod_bottom" site2="left_rodA_plate_target"   solref="0.001 1" solimp="0.999 0.99 0.001"/>
-          <connect name="left_rodB_loop" site1="left_rodB_rod_bottom" site2="left_rodB_plate_target"   solref="0.001 1" solimp="0.999 0.99 0.001"/>
-          <connect name="right_rodA_loop" site1="right_rodA_rod_bottom" site2="right_rodA_plate_target"   solref="0.001 1" solimp="0.999 0.99 0.001"/>
-          <connect name="right_rodB_loop" site1="right_rodB_rod_bottom" site2="right_rodB_plate_target"   solref="0.001 1" solimp="0.999 0.99 0.001"/>
+          <connect name="left_rodA_loop" site1="left_rodA_rod_bottom" site2="left_rodA_plate_target"   solref="0.001 0.5" solimp="0.999 0.99 0.001"/>
+          <connect name="left_rodB_loop" site1="left_rodB_rod_bottom" site2="left_rodB_plate_target"   solref="0.001 0.5" solimp="0.999 0.99 0.001"/>
+          <connect name="right_rodA_loop" site1="right_rodA_rod_bottom" site2="right_rodA_plate_target"   solref="0.001 0.5" solimp="0.999 0.99 0.001"/>
+          <connect name="right_rodB_loop" site1="right_rodB_rod_bottom" site2="right_rodB_plate_target"   solref="0.001 0.5" solimp="0.999 0.99 0.001"/>
         </equality>
         <sensor>
