Commit message: add controllers with ros2 control

File: mujoco_ros2_control_examples/urdf/yaro/mujoco_actuators.urdf.xacro (robot description, xacro)
@@ -30,5 +30,9 @@
        caps a ur10e at 45% of its own, and both errors are silent. -->
   <xacro:property name="yaro_max_effort" value="${dict(
-      yaro_1105     = [ 194,  194,  102,  34,  34,  34])}"/>
+    yaro_1115     = [ 411,  411,  102, 102,  66,  66],
+    yaro_1105     = [ 194,  194,  102,  34,  34,  34],
+    yaro_0808     = [ 194,  194,  102,  34,  34,  34],
+    yaro_1310     = [ 411,  411,  102, 102,  66,  66],
+    yaro_1608     = [ 411,  411,  194, 102,  34,  34])}"/>
   <!-- The gains were tuned on the ur5e, so they are carried to other sizes by
        scaling with each joint's torque: an arm twice as strong gets twice the

File: mujoco_ros2_control_examples/urdf/yaro/ros2_control.urdf.xacro (robot description, xacro)
@@ -1,5 +1,5 @@
 <?xml version="1.0"?>
 <robot xmlns:xacro="http://www.ros.org/wiki/xacro">
-  <xacro:macro name="yaro_1105_ros2_control"
+  <xacro:macro name="yaro_ros2_control"
     params="mujoco
      mujoco_effort

File: mujoco_ros2_control_examples/urdf/yaro/yaro.urdf.xacro (robot description, xacro)
@@ -30,4 +30,6 @@
          neither a window nor a display, so a headless run still produces images. -->
   <xacro:arg name="headless" default="false" />
+  <!-- One of 1115 1105 0808 1310 1608 -->
+  <xacro:arg name="yaro_type" default="$(arg name)" />
   <!-- Import franka urdf file -->
   <link name="world" />
@@ -37,8 +39,8 @@
     <origin rpy="$(arg base_rpy)" xyz="$(arg base_xyz)" />
   </joint>
-  <xacro:include filename="$(find mujoco_ros2_control_examples)/urdf/yaro_1105/yaro_1105.urdf" />
+  <xacro:include filename="$(find mujoco_ros2_control_examples)/urdf/yaro/$(arg yaro_type).urdf" />
   <!-- Import franka ros2_control -->
-  <xacro:include filename="$(find mujoco_ros2_control_examples)/urdf/yaro_1105/ros2_control.urdf.xacro" />
-  <xacro:yaro_1105_ros2_control
+  <xacro:include filename="$(find mujoco_ros2_control_examples)/urdf/yaro/ros2_control.urdf.xacro" />
+  <xacro:yaro_ros2_control
     use_fake_hardware="$(arg use_fake_hardware)"
     fake_sensor_commands="$(arg fake_sensor_commands)"
@@ -48,7 +50,7 @@
   <!-- Configure mujoco -->
   <xacro:if value="$(arg mujoco)">
-    <xacro:include filename="$(find mujoco_ros2_control_examples)/urdf/yaro_1105/mujoco_actuators.urdf.xacro" />
+    <xacro:include filename="$(find mujoco_ros2_control_examples)/urdf/yaro/mujoco_actuators.urdf.xacro" />
     <mujoco>
-      <xacro:create_mujoco_actuators tf_prefix="" yaro_type="yaro_1105"/>
+      <xacro:create_mujoco_actuators tf_prefix="" yaro_type="$(arg yaro_type)"/>
       <compiler meshdir="$(arg mujoco_model_path)/meshes"
         discardvisual="false"
